File: IR-Digipot/Hardware/Power.sch (KiCad schematic (older format))
At the start: 40 parts, among them Q7 STL6P3LLH6, U8 L7985TR, U9 LM27761

Commit message: Wire high-side switch FET for +5VA
The PIC port should be able to draw enough current to
properly control the switch.
Connections:
- net +5VA_SHTDN: now reaches R36.1
Changed lines of the file:
@@
 Wire Wire Line
 	10050 4100 10050 4300
+Text GLabel 1450 4950 0    50   Input ~ 0
++5VA_SHTDN
+Wire Wire Line
+	1450 4950 1550 4950
+Wire Wire Line
+	1550 4950 1550 4850
 $EndSCHEMATC

Commit message: Tweak digipot preamp gain
Allows to feed professional equipment level of signal which is
3.472 Vpp. There is enough swing to do 4 Vpp with the new gain.
Parts:
- renumbered C31 to C32, C32 to C33, C41 to C34, C33 to C35, C34 to C36, C42 to C37, C43 to C38, C35 to C39, C36 to C40, C37 to C41, C44 to C42, C45 to C43, C46 to C44, C38 to C45, C47 to C46, C39 to C47, C40 to C48, C48 to C49, FB3 to FB2, FB2 to FB3, L3 to L1, L1 to L2, L2 to L3, R35 to R33, R36 to R34, R38 to R35, R37 to R36, R31 to R37, R32 to R38, R33 to R39, R34 to R40, R39 to R41, R40 to R42, R41 to R43
Other:
- note added: "Switch for +5v in analog circuits"
- note removed: "Switch for +%v in analog circuits"

Commit message: Add status LEDs to the digipot
Parts:
- renumbered D8 to D10, D7 to D9, R33 to R35, R34 to R36, R35 to R37, R36 to R38, R37 to R39, R38 to R40, R39 to R41, R40 to R42, R41 to R43, R42 to R44, R43 to R45

Commit message: Refactor library
Split it into smaller files, which contains components related to each
other.

The goal is to make the library reusable across projects.

The resistors and capacitors are still only generic symbols in the
library and it is still up to designer to link to DigiKey. With time
those components will become accessible via library as well.
Parts:
- C32: footprint Librray:C_1210_3225Metric -> Capacitor_Ceramic:C_1210_3225Metric; symbol Library:C -> Capacitor_Ceramic:C
- C33, C46: footprint Librray:C_0603_1608Metric -> Capacitor_Ceramic:C_0603_1608Metric; symbol Library:C -> Capacitor_Ceramic:C
- C34, C35, C36, C37, C38, C39, C43, C45, C47, C49: footprint Librray:C_0402_1005Metric -> Capacitor_Ceramic:C_0402_1005Metric; symbol Library:C -> Capacitor_Ceramic:C
- C40, C41, C42, C44, C48: footprint Librray:C_0805_2012Metric -> Capacitor_Ceramic:C_0805_2012Metric; symbol Library:C -> Capacitor_Ceramic:C
- D10: footprint Librray:D_0603_1610Metric -> Diode:D_0603_1610Metric; symbol Library:D_ZENNER -> Diode:D_ZENNER
- D9: footprint Librray:SOD-323HE -> Diode:SOD-323HE; symbol Library:D_SCHOTTKY -> Diode:D_SCHOTTKY
- FB2, FB3, FB4: value Ferrite_Bead -> BLM15PG100SN1D; footprint Librray:L_0402_1005Metric -> Inductor:L_0402_1005Metric; symbol Library:Ferrite_Bead -> Inductor:BLM15PG100SN1D; Detailed Description (none) -> 10 Ohms @ 100MHz 1 Power Line Ferrite Bead 0402 (1005 Metri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
- L1, L3: value ACP3225 -> ACP3225-102-2P-T000; footprint Librray:ACP3225 -> Inductor:ACP3225; symbol Library:EMI_Filter_CommonMode -> Inductor:ACP3225-102-2P-T000; Detailed Description (none) -> 2 Line Common Mode Choke Surface Mount 1 kOhms @ 100MHz 1.5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
- L2: value 22uH -> LQH44PN220MP0L; footprint Librray:L_1515_4040Metric -> Inductor:L_1515_4040Metric; symbol Library:INDUCTOR -> Inductor:LQH44PN220MP0L; Detailed Description (none) -> 22µH Shielded Wirewound Inductor 790mA 444mOhm Max Nonstand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; Inductance (none) -> 22µH
- Q7: footprint Librray:8-PowerVDFN -> Package_DFN_QFN:8-PowerVDFN; symbol Library:P-CHANNEL-SGD -> Transistor_FET:STL6P3LLH6; Detailed Description (none) -> P-Channel 30V 6A (Tc) 2.9W (Tc) Surface Mount PowerFlat™ (3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
- R35, R36, R37, R38, R39, R40, R41, R42, R43, R44, R45: footprint Librray:R_0402_1005Metric -> Resistor:R_0402_1005Metric; symbol Library:R -> Resistor:R
- U8: footprint Librray:VFDFPN-10_EP_3x3mm_P0.5mm -> Package_DFN_QFN:VFDFPN-10_EP_3x3mm_P0.5mm; symbol Library:L7985TR -> Power_Management:L7985TR; Detailed Description (none) -> Buck Switching Regulator IC Positive Adjustable 0.6V 1 Outp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
- U9: value LM27761 -> LM27761DSGR; footprint Librray:WSON-8-EP_P0.5mm -> Package_SON:WSON-8-EP_P0.5mm; symbol Library:LM27761 -> Power_Management:LM27761DSGR; Detailed Description (none) -> Charge Pump Switching Regulator IC Negative Adjustable -1.5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
