File: IR-Digipot/Hardware/IR Digipot.kicad_pcb (KiCad board)
At the start: 2 copper layers, 54.6 x 58.4 mm, 126 parts, among them J1 Conn_1x06_Generic, J2 Conn_1x03_Generic, J3 STX-3500-5NTR, J4 STX-3500-5NTR, J5 Molex_1054500101, Q1 MMBT3904, Q2 MMBT3906, Q3 MMBT3904, Q4 MMBT3906, Q5 STL6P3LLH6, Q6 STL6P3LLH6, Q7 STL6P3LLH6, U1 PIC18F2550T-I/SO, U2 TCM809, U3 TSOP754, U4 AD5262, U5 OPA2134, U6 OPA2134, U7 STUSB4500QTR, U8 L7985TR, U9 LM27761, X1 20 MHz

Commit message: Wire high-side switch FET for +5VA
The PIC port should be able to draw enough current to
properly control the switch.
Connections:
- R36 pad 1: Net-(R36-Pad1) -> +5VA_SHTDN
- U1 pad 6: Net-(U1-Pad6) -> +5VA_SHTDN

Commit message: Continue routing digipot receiver
Minor touches to the USB-C PD tracks, routed signal paths of
audio circuits.

Added missing reset circuits for the digipot.
Parts:
- added C49: 0.1uF, Librray:C_0402_1005Metric, F.Cu at (127.8, 124.0)
- added R42: 3.3K, Librray:R_0402_1005Metric, F.Cu at (127.8, 122.8)
- moved C29 6.29 mm to (150.7, 82.7), turned to 180 degrees
- moved D5 2.47 mm to (150.8, 81.5), turned to 180 degrees
- moved C39 1.85 mm to (140.1, 89.9)
- moved C32 1.65 mm to (140.9, 77.9), turned to 0 degrees
- moved C40 1.19 mm to (138.7, 89.5)
- moved Q7 1.05 mm to (139.8, 94.7)
- moved R35 1.05 mm to (140.1, 97.2)
- moved R36 1.05 mm to (140.1, 98.1)
- moved R38 1.05 mm to (137.2, 95.7)
- moved C41 1.05 mm to (142.4, 93.7)
- moved R37 1.05 mm to (142.4, 95.6)
- moved R32 0.95 mm to (145.2, 79.9)
- moved R33 0.95 mm to (145.2, 80.8)
- moved L3 0.92 mm to (145.4, 94.6)
- moved FB3 0.92 mm to (144.3, 97.6)
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Connections:
- J3 pad 4: Net-(J3-Pad4) -> GNDA
- J3 pad 5: Net-(J3-Pad5) -> GNDA
- J4 pad 4: Net-(J4-Pad4) -> GNDA
- J4 pad 5: Net-(J4-Pad5) -> GNDA
- U1 pad 5: DIGIPOT_SHDN -> +5VA_SHTDN
- U1 pad 6: +5VA_SHTDN -> DIGIPOT_SHDN
Routing:
- net VBUS: track 0.00 -> 36.1 mm
- net GNDA: track 0.00 -> 35.3 mm, vias 0 -> 2
- net /Audio/AUDIO_RIGHT_IN: track 0.00 -> 31.0 mm
- net GND: track 0.00 -> 24.6 mm, vias 0 -> 9
- net Net-(J1-Pad5): track 0.00 -> 22.4 mm
- net Net-(C18-Pad2): track 0.00 -> 21.9 mm
- net Net-(J1-Pad4): track 0.00 -> 21.6 mm
- net VSNK: track 0.00 -> 21.2 mm
- net Net-(C17-Pad2): track 0.00 -> 19.3 mm
- net /Audio/AUDIO_RIGHT_OUT: track 0.00 -> 18.1 mm
- net /Audio/AUDIO_LEFT_OUT: track 0.00 -> 17.9 mm
- net /Audio/AUDIO_LEFT_IN: track 0.00 -> 17.5 mm
- net /CPU/IR_SERIAL: track 0.00 -> 16.7 mm
- net Net-(D4-Pad2): track 0.00 -> 12.0 mm
- net Net-(D4-Pad1): track 0.00 -> 11.3 mm
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- added copper zone on F.Cu, net GND
Other:
- net class Default: via_dia 0.2032 -> 0.508; via_drill 0.1524 -> 0.3048

Commit message: Remove connection from audio jacks switches
Were wrongly connected to ground. The idea was to connect
unused pads to big copper mass to give mechanical rigidity.

Should be done using non-connected net.
Connections:
- J3 pad 4: GNDA -> Net-(J3-Pad4)
- J3 pad 5: GNDA -> Net-(J3-Pad5)
- J4 pad 4: GNDA -> Net-(J4-Pad4)
- J4 pad 5: GNDA -> Net-(J4-Pad5)

Commit message: Fully routed USB-C PD and +5VD regulators
Zones will need some tweaks, but electrically those circuits
are usable now.
Parts:
- moved D6 51.1 mm to (113.6, 95.1), turned to 90 degrees
- moved C30 49.0 mm to (114.8, 95.2), turned to 270 degrees
- moved R28 47.6 mm to (114.8, 93.2), turned to 90 degrees
- moved R22 43.3 mm to (116.1, 89.6), turned to 0 degrees
- moved Q6 43.3 mm to (117.5, 94.1), turned to 180 degrees
- moved R19 43.0 mm to (116.1, 88.7), turned to 0 degrees
- moved R21 42.7 mm to (116.1, 86.9), turned to 0 degrees
- moved R20 42.6 mm to (116.1, 87.8), turned to 0 degrees
- moved R29 42.6 mm to (116.1, 86.0), turned to 180 degrees
- moved R23 42.6 mm to (116.1, 85.2), turned to 0 degrees
- moved R27 41.5 mm to (117.5, 91.5), turned to 0 degrees
- moved J5 41.5 mm to (117.7, 79.0), turned to 270 degrees
- moved R26 41.0 mm to (117.5, 90.6), turned to 180 degrees
- moved C25 39.0 mm to (120.1, 76.5), turned to 270 degrees
- moved Q5 35.4 mm to (121.9, 94.1), turned to 180 degrees
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Connections:
- L2 pad 1: GND -> /Power/+5V_UNFILTERED
- L2 pad 2: GNDD -> Net-(C38-Pad2)
- L2 pad 3: /Power/+5V_UNFILTERED -> GND
- L2 pad 4: Net-(C38-Pad2) -> GNDD
Routing:
- net VSNK: track 21.2 -> 64.1 mm, vias 0 -> 3
- net GND: track 24.6 -> 50.1 mm, vias 9 -> 29
- net +2V7: track 1.75 -> 14.2 mm, vias 0 -> 2
- net /Power/+5V_UNFILTERED: track 7.32 -> 16.3 mm
- net /CPU/IR_SERIAL: track 16.7 -> 25.7 mm
- net Net-(C26-Pad2): track 10.8 -> 18.7 mm, vias 0 -> 2
- net Net-(D7-Pad1): track 5.80 -> 9.33 mm
- net Net-(C33-Pad2): track 0.95 -> 2.80 mm
- net Net-(C33-Pad1): track 4.06 -> 5.77 mm
- net VBUS: track 36.1 -> 37.4 mm
- net Net-(R20-Pad2): track 1.93 -> 2.82 mm
- net Net-(R29-Pad1): track 1.39 -> 2.23 mm
- added copper zone on B.Cu, net GND

Commit message: Return USB-C connector to proper side
Some of the grounds are now disconnected, will be connected back as part
of zones rework.
Parts:
- moved D6 52.1 mm to (161.1, 73.6), turned to 270 degrees
- moved C30 50.0 mm to (159.9, 73.5), turned to 90 degrees
- moved R28 48.4 mm to (159.9, 75.6), turned to 270 degrees
- moved Q6 44.3 mm to (157.3, 74.6), turned to 0 degrees
- moved R22 43.9 mm to (158.7, 79.1), turned to 180 degrees
- moved R19 43.5 mm to (158.7, 80.0), turned to 180 degrees
- moved R20 43.1 mm to (158.6, 80.9), turned to 180 degrees
- moved R21 42.9 mm to (158.6, 81.8), turned to 180 degrees
- moved R29 42.7 mm to (158.6, 82.7), turned to 0 degrees
- moved R23 42.6 mm to (158.7, 83.6), turned to 180 degrees
- moved R27 42.3 mm to (157.3, 77.2), turned to 180 degrees
- moved R26 41.7 mm to (157.3, 78.1), turned to 0 degrees
- moved J5 40.8 mm to (157.0, 89.7), turned to 90 degrees
- moved C25 37.9 mm to (154.6, 92.2), turned to 90 degrees
- moved Q5 36.7 mm to (152.9, 74.6), turned to 0 degrees
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Routing:
- net /CPU/IR_SERIAL: track 25.7 -> 14.1 mm
- net GND: track 50.1 -> 39.2 mm
- net VSNK: track 64.1 -> 56.8 mm, vias 3 -> 4

Commit message: Rework power supply ground zones
USB-C PD and +5VD regulator can now be considered final: small tweaks
are possible, but overall seems all fine.
Parts:
- moved C40 7.78 mm to (137.6, 89.2), turned to 90 degrees
- moved C39 5.12 mm to (139.0, 89.0), turned to 90 degrees
- moved FB2 5.01 mm to (139.5, 90.4), turned to 180 degrees
- moved C38 3.09 mm to (140.0, 89.0), turned to 270 degrees
- moved L2 1.35 mm to (141.9, 88.9), turned to 270 degrees
- moved J5 0.51 mm to (157.0, 90.2)
- moved C25 0.51 mm to (154.6, 92.7)
- moved C26 0.51 mm to (150.6, 84.1)
- moved D5 0.51 mm to (150.9, 79.6)
- moved R19 0.51 mm to (158.7, 80.5)
- moved R23 0.51 mm to (158.7, 84.1)
- moved R24 0.51 mm to (150.7, 78.6)
- moved R25 0.51 mm to (152.7, 78.6)
- moved R26 0.51 mm to (157.3, 78.6)
- moved R29 0.51 mm to (158.6, 83.2)
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Connections:
- L2 pad 1: /Power/+5V_UNFILTERED -> GND
- L2 pad 2: Net-(C38-Pad2) -> GNDD
- L2 pad 3: GND -> /Power/+5V_UNFILTERED
- L2 pad 4: GNDD -> Net-(C38-Pad2)
Routing:
- net VSNK: track 56.8 -> 52.2 mm, vias 4 -> 2
- net GND: track 39.2 -> 35.1 mm, vias 29 -> 24
- net /Power/+5V_UNFILTERED: track 16.3 -> 14.0 mm
- net GNDD: track 10.3 -> 11.3 mm, vias 0 -> 4
- added copper zone on B.Cu, net GNDD
- added copper zone on F.Cu, net GNDD
- added copper zone on F.Cu, net Net-(D7-Pad1)
Other:
- board size 54.6 x 58.4 mm -> 54.9 x 58.4 mm

Commit message: Route microcontroller area
Routing:
- net +5VD: track 9.45 -> 61.3 mm, vias 0 -> 2
- net +5VA_SHTDN: track 0.00 -> 26.1 mm
- net Net-(J2-Pad2): track 0.00 -> 18.5 mm, vias 0 -> 1
- net Net-(J2-Pad1): track 0.00 -> 15.3 mm, vias 0 -> 1
- net GNDD: track 11.3 -> 20.0 mm, vias 4 -> 11

Commit message: Finish routing IR digipot
All nets are routed, no DRC errors reported.

Next steps are to do little tweaks to topology to minimize track
length, double-check the design and capabilities of the PCB house.
Parts:
- moved C44 2.41 mm to (135.7, 105.5)
- moved C45 2.41 mm to (136.1, 100.1)
- moved FB4 2.41 mm to (139.9, 105.0)
- moved R39 2.41 mm to (139.9, 101.1)
- moved R41 2.41 mm to (139.9, 103.0)
- moved U9 2.41 mm to (137.2, 102.1)
- moved C46 2.41 mm to (137.5, 105.5)
- moved C47 2.41 mm to (138.8, 103.6)
- moved C48 2.41 mm to (140.4, 106.3)
- moved R40 2.41 mm to (138.8, 101.1)
- moved C5 0.66 mm to (131.2, 112.5), turned to 180 degrees
- moved C7 0.66 mm to (132.0, 113.9), turned to 180 degrees
Routing:
- net +5VA: track 10.2 -> 101.2 mm, vias 0 -> 6
- net -5VA: track 6.50 -> 91.1 mm, vias 0 -> 8
- net DIGIPOT_SHDN: track 0.00 -> 37.4 mm, vias 0 -> 2
- net SPI_CS_DIGIPOT: track 0.00 -> 29.2 mm, vias 0 -> 2
- net SPI_MOSI: track 0.00 -> 23.1 mm, vias 0 -> 2
- net SPI_CLK: track 0.00 -> 22.3 mm, vias 0 -> 2
- net GNDA: track 35.3 -> 50.2 mm, vias 2 -> 34
- net /Audio/AUDIO_RIGHT_PREAMP: track 2.99 -> 16.2 mm
- net /Audio/AUDIO_LEFT_PREAMP: track 2.99 -> 11.9 mm
- net /Audio/AUDIO_RIGHT_ATT: track 4.68 -> 6.76 mm
- net Net-(FB1-Pad2): track 4.30 -> 4.87 mm
- net VSNK: track 52.2 -> 51.7 mm
- added copper zone on F.Cu, net +5VA
- added copper zone on F.Cu, net -5VA
- added copper zone on B.Cu, net GNDA
- added copper zone on F.Cu, net GNDA
- added copper zone on F.Cu, net Net-(J3-Pad4)
- added copper zone on F.Cu, net Net-(J3-Pad5)
- added copper zone on F.Cu, net Net-(J4-Pad4)
- added copper zone on F.Cu, net Net-(J4-Pad5)
