File: IR-Digipot/Hardware/IR Digipot.kicad_pcb (KiCad board)
At the start: 2 copper layers, 54.9 x 58.4 mm, 128 parts, among them J1 Conn_1x06_Generic, J2 Conn_1x03_Generic, J3 STX-3500-5NTR, J4 STX-3500-5NTR, J5 Molex_1054500101, Q1 MMBT3904, Q2 MMBT3906, Q3 MMBT3904, Q4 MMBT3906, Q5 STL6P3LLH6, Q6 STL6P3LLH6, Q7 STL6P3LLH6, U1 PIC18F2550T-I/SO, U2 TCM809, U3 TSOP754, U4 AD5262, U5 OPA2134, U6 OPA2134, U7 STUSB4500QTR, U8 L7985TR, U9 LM27761, X1 20 MHz

Commit message: Swap MOSI and CS uC pins
Allows to route tracks more efficiently.
Connections:
- R3 pad 2: SPI_CS_DIGIPOT -> SPI_MOSI
- R4 pad 2: SPI_MOSI -> SPI_CS_DIGIPOT
Routing:
- net SPI_CS_DIGIPOT: track 29.2 -> 26.7 mm
- net SPI_MOSI: track 23.1 -> 22.6 mm
Changed lines of the file:
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@@
     (thickness 1.6)
     (drawings 48)
-    (tracks 862)
+    (tracks 856)
     (zones 0)
     (modules 128)
@@
     (fp_line (start 0.889 0.381) (end 0.889 -0.381) (layer F.CrtYd) (width 0.12))
     (pad 2 smd rect (at 0.508 0 270) (size 0.6 0.7) (layers F.Cu F.Paste F.Mask)
-      (net 34 SPI_MOSI))
+      (net 33 SPI_CS_DIGIPOT))
     (pad 1 smd rect (at -0.508 0 270) (size 0.6 0.7) (layers F.Cu F.Paste F.Mask)
       (net 31 "Net-(R4-Pad1)"))
@@
     (fp_line (start 0.889 0.381) (end 0.889 -0.381) (layer F.CrtYd) (width 0.12))
     (pad 2 smd rect (at 0.508 0 270) (size 0.6 0.7) (layers F.Cu F.Paste F.Mask)
-      (net 33 SPI_CS_DIGIPOT))
+      (net 34 SPI_MOSI))
     (pad 1 smd rect (at -0.508 0 270) (size 0.6 0.7) (layers F.Cu F.Paste F.Mask)
       (net 30 "Net-(R3-Pad1)"))
@@
   (via (at 129.8448 120.0404) (size 0.508) (drill 0.3048) (layers F.Cu B.Cu) (net 33))
   (via (at 130.4544 110.236) (size 0.508) (drill 0.3048) (layers F.Cu B.Cu) (net 32))
-  (via (at 129.794 110.236) (size 0.508) (drill 0.3048) (layers F.Cu B.Cu) (net 33))
-  (via (at 129.1336 110.236) (size 0.508) (drill 0.3048) (layers F.Cu B.Cu) (net 34))
+  (via (at 129.794 110.236) (size 0.508) (drill 0.3048) (layers F.Cu B.Cu) (net 34))
+  (via (at 129.1336 110.236) (size 0.508) (drill 0.3048) (layers F.Cu B.Cu) (net 33))
   (via (at 131.1656 116.586) (size 0.508) (drill 0.3048) (layers F.Cu B.Cu) (net 35))
   (via (at 130.5052 116.586) (size 0.508) (drill 0.3048) (layers F.Cu B.Cu) (net 32))
@@
   (segment (start 129.8685 120.0641) (end 129.8448 120.0404) (width 0.3048) (layer F.Cu) (net 33))
   (segment (start 129.8685 121.264) (end 129.8685 120.0641) (width 0.3048) (layer F.Cu) (net 33))
-  (segment (start 129.54 109.5248) (end 129.794 109.7788) (width 0.4064) (layer B.Cu) (net 33))
-  (segment (start 128.778 109.5248) (end 129.54 109.5248) (width 0.4064) (layer B.Cu) (net 33))
-  (segment (start 128.3208 112.9792) (end 128.3208 109.982) (width 0.4064) (layer B.Cu) (net 33))
-  (segment (start 129.1844 113.8428) (end 128.3208 112.9792) (width 0.4064) (layer B.Cu) (net 33))
-  (segment (start 129.1844 119.38) (end 129.1844 113.8428) (width 0.4064) (layer B.Cu) (net 33))
-  (segment (start 129.794 109.7788) (end 129.794 110.236) (width 0.4064) (layer B.Cu) (net 33))
-  (segment (start 128.3208 109.982) (end 128.778 109.5248) (width 0.4064) (layer B.Cu) (net 33))
-  (segment (start 129.8448 120.0404) (end 129.1844 119.38) (width 0.4064) (layer B.Cu) (net 33))
-  (segment (start 129.794 99.06) (end 129.794 110.236) (width 0.4064) (layer F.Cu) (net 33))
-  (segment (start 127.3302 96.5962) (end 129.794 99.06) (width 0.4064) (layer F.Cu) (net 33))
-  (segment (start 127.3302 96.1898) (end 127.3302 96.5962) (width 0.4064) (layer F.Cu) (net 33))
+  (segment (start 129.794 99.06) (end 129.794 110.236) (width 0.4064) (layer F.Cu) (net 34))
+  (segment (start 127.3302 96.5962) (end 129.794 99.06) (width 0.4064) (layer F.Cu) (net 34))
+  (segment (start 127.3302 96.1898) (end 127.3302 96.5962) (width 0.4064) (layer F.Cu) (net 34))
   (segment (start 129.8685 115.464) (end 129.8685 116.5623) (width 0.3048) (layer F.Cu) (net 34))
   (segment (start 129.8685 116.5623) (end 129.8448 116.586) (width 0.3048) (layer F.Cu) (net 34))
   (via (at 129.8448 116.586) (size 0.508) (drill 0.3048) (layers F.Cu B.Cu) (net 34))
-  (segment (start 129.1336 112.5728) (end 129.1336 110.236) (width 0.4064) (layer B.Cu) (net 34))
-  (segment (start 129.8448 113.284) (end 129.1336 112.5728) (width 0.4064) (layer B.Cu) (net 34))
-  (segment (start 129.8448 116.586) (end 129.8448 113.284) (width 0.4064) (layer B.Cu) (net 34))
-  (segment (start 129.1336 99.6188) (end 129.1336 110.236) (width 0.4064) (layer F.Cu) (net 34))
-  (segment (start 126.0602 96.5454) (end 129.1336 99.6188) (width 0.4064) (layer F.Cu) (net 34))
-  (segment (start 126.0602 96.1898) (end 126.0602 96.5454) (width 0.4064) (layer F.Cu) (net 34))
+  (segment (start 129.1336 99.6188) (end 129.1336 110.236) (width 0.4064) (layer F.Cu) (net 33))
+  (segment (start 126.0602 96.5454) (end 129.1336 99.6188) (width 0.4064) (layer F.Cu) (net 33))
+  (segment (start 126.0602 96.1898) (end 126.0602 96.5454) (width 0.4064) (layer F.Cu) (net 33))
+  (segment (start 129.1844 110.2868) (end 129.1336 110.236) (width 0.4064) (layer B.Cu) (net 33))
+  (segment (start 129.1844 119.38) (end 129.1844 110.2868) (width 0.4064) (layer B.Cu) (net 33))
+  (segment (start 129.8448 120.0404) (end 129.1844 119.38) (width 0.4064) (layer B.Cu) (net 33))
+  (segment (start 129.8448 110.2868) (end 129.794 110.236) (width 0.4064) (layer B.Cu) (net 34))
+  (segment (start 129.8448 116.586) (end 129.8448 110.2868) (width 0.4064) (layer B.Cu) (net 34))
   (segment (start 131.1685 116.5831) (end 131.1656 116.586) (width 0.3048) (layer F.Cu) (net 35))
   (segment (start 131.1685 115.464) (end 131.1685 116.5831) (width 0.3048) (layer F.Cu) (net 35))
@@
     (polygon
       (pts
-        (xy 129.286 129.54) (xy 128.524 129.54) (xy 128.524 110.236) (xy 129.286 110.236)
-      )
-    )
-  )
-  (zone (net 0) (net_name "") (layer B.Cu) (hatch none 0.508)
-    (connect_pads yes (clearance 0.254))
-    (min_thickness 0.254)
-    (keepout (tracks allowed) (vias allowed) (copperpour not_allowed))
-    (fill (arc_segments 32) (thermal_gap 0.254) (thermal_bridge_width 0.508))
-    (polygon
-      (pts
         (xy 136.144 129.54) (xy 135.128 129.54) (xy 135.128 110.236) (xy 136.144 110.236)
       )
@@
       )
     )
+  )
+  (zone (net 0) (net_name "") (layer B.Cu) (hatch none 0.508)
+    (connect_pads yes (clearance 0.254))
+    (min_thickness 0.254)
+    (keepout (tracks allowed) (vias allowed) (copperpour not_allowed))
+    (fill (arc_segments 32) (thermal_gap 0.254) (thermal_bridge_width 0.508))
+    (polygon
+      (pts
+        (xy 129.286 129.54) (xy 128.524 129.54) (xy 128.524 110.236) (xy 129.286 110.236)
+      )
+    )

Commit message: Prevision digipot power from +5VD
The idea is to try to bring digipot running before powering on
buffers with the goal of programming proper volume on power on.

Should help reducing popping on power on.
Parts:
- added R43: NC, Librray:R_0402_1005Metric, F.Cu at (135.5, 119.1)
- moved FB1 1.52 mm to (135.5, 117.1)
- moved R42 1.14 mm to (127.7, 124.0)
- moved C49 1.12 mm to (127.7, 122.8)
- moved C20 1.04 mm to (136.6, 115.2), turned to 90 degrees
Connections:
- FB1 pad 2: Net-(FB1-Pad2) -> /Audio/DIGIPOT_VL
- R42 pad 1: +5VA -> /Audio/DIGIPOT_VL
- U4 pad 13: Net-(FB1-Pad2) -> /Audio/DIGIPOT_VL
Routing:
- net +5VD: track 61.3 -> 93.0 mm, vias 2 -> 6
- net /Audio/DIGIPOT_VL: track 0.00 -> 17.1 mm
- net Net-(FB1-Pad2): track 4.87 -> 0.00 mm
- net GNDA: track 50.2 -> 51.5 mm
- net -5VA: track 91.1 -> 92.0 mm

Commit message: Add revision and date to the board
Other:
- board text added: "IR-Digipot"
- board text added: "Jan, 2021"
- board text added: "Rev.A"
Changed lines of the file:
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@@
   (general
     (thickness 1.6)
-    (drawings 48)
+    (drawings 51)
     (tracks 881)
     (zones 0)
@@
     )
   )
+  (gr_text "Jan, 2021" (at 113.5888 128.3208) (layer F.SilkS)
+    (effects (font (size 0.6096 0.6096) (thickness 0.1524)) (justify left))
+  )
+  (gr_text Rev.A (at 110.5916 128.3208) (layer F.SilkS)
+    (effects (font (size 0.6096 0.6096) (thickness 0.1524)) (justify left))
+  )
+  (gr_text IR-Digipot (at 110.5916 127.3556) (layer F.SilkS)
+    (effects (font (size 0.6096 0.6096) (thickness 0.1524)) (justify left))
+  )
   (gr_line (start 164.592 129.54) (end 109.728 129.54) (layer Edge.Cuts) (width 0.05))

Commit message: Tweak digipot preamp gain
Allows to feed professional equipment level of signal which is
3.472 Vpp. There is enough swing to do 4 Vpp with the new gain.
Parts:
- R10: renamed from R8; value 3.3K -> 12K
- R13: renamed from R15; value 3.3K -> 12K
- R14: renamed from R16; value 3.3K -> 12K
- R17: renamed from R11; value 33K -> 22K
- R18: renamed from R12; value 33K -> 22K
- R7: renamed from R13; value 33K -> 22K
- R8: renamed from R14; value 33K -> 22K
- R9: renamed from R7; value 3.3K -> 12K
- renumbered C2 to C1, C17 to C11, C18 to C12, C11 to C13, C12 to C14, C23 to C15, C24 to C16, C21 to C17, C22 to C18, C15 to C19, C3 to C2, C16 to C20, C5 to C21, C6 to C22, C49 to C23, C7 to C24, C8 to C25, C25 to C26, C29 to C27, C26 to C28, C27 to C29, C1 to C3, C28 to C30, C30 to C31, C31 to C32, C32 to C33, C41 to C34, C33 to C35, C34 to C36, C42 to C37, C43 to C38, C35 to C39, C36 to C40, C37 to C41, C44 to C42, C45 to C43, C46 to C44, C38 to C45, C47 to C46, C39 to C47, C40 to C48, C48 to C49, C19 to C5, C20 to C6, C13 to C7, C14 to C8, FB3 to FB2, FB2 to FB3, L3 to L1, L1 to L2, L2 to L3, R9 to R11, R10 to R12, R17 to R15, R18 to R16, R42 to R19, R43 to R20, R19 to R21, R20 to R22, R21 to R23, R22 to R26, R26 to R27, R30 to R28, R27 to R29, R23 to R30, R28 to R31, R29 to R32, R35 to R33, R36 to R34, R38 to R35, R37 to R36, R31 to R37, R32 to R38, R33 to R39, R34 to R40, R39 to R41, R40 to R42, R41 to R43, U2 to U1, U1 to U2, U6 to U4, U4 to U6

Commit message: Add status LEDs to the digipot
Parts:
- added D1: HSMG-C170, Librray:HSMx-C170, F.Cu at (118.7, 74.3)
- added D2: HSMG-C170, Librray:HSMx-C170, F.Cu at (120.7, 74.3)
- added R5: 150, Librray:R_0402_1005Metric, F.Cu at (122.7, 76.5)
- added R6: 150, Librray:R_0402_1005Metric, F.Cu at (122.7, 75.6)
- renumbered D8 to D10, D1 to D3, D2 to D4, D3 to D5, D4 to D6, D5 to D7, D6 to D8, D7 to D9, R8 to R10, R9 to R11, R10 to R12, R11 to R13, R12 to R14, R13 to R15, R14 to R16, R15 to R17, R16 to R18, R17 to R19, R18 to R20, R19 to R21, R20 to R22, R21 to R23, R22 to R24, R23 to R25, R24 to R26, R25 to R27, R26 to R28, R27 to R29, R28 to R30, R29 to R31, R30 to R32, R31 to R33, R32 to R34, R33 to R35, R34 to R36, R35 to R37, R36 to R38, R37 to R39, R38 to R40, R39 to R41, R40 to R42, R41 to R43, R42 to R44, R43 to R45, R5 to R7, R6 to R8, R7 to R9
Connections:
- U2 pad 2: Net-(U2-Pad2) -> /CPU/LED0
- U2 pad 3: Net-(U2-Pad3) -> /CPU/LED1
Routing:
- net /CPU/LED1: track 0.00 -> 8.13 mm
- net /CPU/LED0: track 0.00 -> 5.38 mm
- net Net-(D1-Pad2): track 0.00 -> 3.89 mm
- net GNDD: track 20.0 -> 22.2 mm, vias 11 -> 13
- net Net-(D2-Pad2): track 0.00 -> 1.62 mm

Commit message: Tweak star ground of digipot
Routing:
- net +5VA: track 100.7 -> 100.1 mm
Changed lines of the file:
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@@
   )
   (setup
-    (last_trace_width 0.4064)
+    (last_trace_width 0.6096)
     (user_trace_width 0.2032)
     (user_trace_width 0.3048)
@@
   (segment (start 144.6149 97.5741) (end 145.1102 97.5741) (width 0.6096) (layer F.Cu) (net 11))
   (segment (start 144.0942 97.5741) (end 144.6149 97.5741) (width 0.6096) (layer F.Cu) (net 11))
-  (segment (start 143.8148 99.06) (end 134.62 99.06) (width 0.6096) (layer B.Cu) (net 11))
-  (segment (start 144.5641 98.3107) (end 143.8148 99.06) (width 0.6096) (layer B.Cu) (net 11))
   (segment (start 131.8185 115.464) (end 131.8185 114.8005) (width 0.3048) (layer F.Cu) (net 11))
   (segment (start 131.4704 114.4524) (end 131.4704 113.919) (width 0.3048) (layer F.Cu) (net 11))
@@
   (segment (start 130.2004 113.3348) (end 130.2004 112.522) (width 0.6096) (layer F.Cu) (net 11))
   (segment (start 130.7846 113.919) (end 130.2004 113.3348) (width 0.6096) (layer F.Cu) (net 11))
-  (segment (start 134.62 99.06) (end 133.4008 100.2792) (width 0.6096) (layer B.Cu) (net 11))
-  (segment (start 133.4008 118.11) (end 133.4008 100.2792) (width 0.6096) (layer B.Cu) (net 11))
   (segment (start 130.2004 112.522) (end 130.2004 111.76) (width 0.6096) (layer F.Cu) (net 11))
   (segment (start 130.2004 111.76) (end 130.556 111.4044) (width 0.6096) (layer F.Cu) (net 11))
@@
   (segment (start 138.6332 118.872) (end 136.3472 116.586) (width 0.6096) (layer F.Cu) (net 11))
   (segment (start 136.3472 116.586) (end 135.4836 116.586) (width 0.6096) (layer F.Cu) (net 11))
+  (segment (start 135.636 99.06) (end 143.8148 99.06) (width 0.6096) (layer B.Cu) (net 11))
+  (segment (start 133.4008 101.2952) (end 135.636 99.06) (width 0.6096) (layer B.Cu) (net 11))
+  (segment (start 143.8148 99.06) (end 144.5641 98.3107) (width 0.6096) (layer B.Cu) (net 11))
+  (segment (start 133.4008 118.11) (end 133.4008 101.2952) (width 0.6096) (layer B.Cu) (net 11))
   (via (at 122.8344 115.0112) (size 0.508) (drill 0.3048) (layers F.Cu B.Cu) (net 12))
   (via (at 132.588 123.2916) (size 0.508) (drill 0.3048) (layers F.Cu B.Cu) (net 12))
@@
     (polygon
       (pts
-        (xy 142.748 99.568) (xy 134.112 99.568) (xy 134.112 108.712) (xy 143.256 108.712) (xy 143.256 100.584)
-        (xy 143.51 100.584) (xy 143.51 108.966) (xy 133.858 108.966) (xy 133.858 99.314) (xy 142.748 99.314)
+        (xy 134.747 100.33) (xy 134.112 100.33) (xy 134.112 108.712) (xy 143.256 108.712) (xy 143.256 101.092)
+        (xy 143.51 101.092) (xy 143.51 108.966) (xy 133.858 108.966) (xy 133.858 100.076) (xy 134.747 100.076)
       )
     )
@@
     (polygon
       (pts
-        (xy 121.412 129.54) (xy 120.904 129.54) (xy 120.904 110.236) (xy 121.412 110.236)
+        (xy 121.158 129.54) (xy 120.904 129.54) (xy 120.904 110.236) (xy 121.158 110.236)
       )
     )
@@
       )
     )
+  )
+  (zone (net 0) (net_name "") (layer B.Cu) (hatch edge 0.508)
+    (connect_pads (clearance 0.254))
+    (min_thickness 0.254)
+    (keepout (tracks not_allowed) (vias not_allowed) (copperpour not_allowed))
+    (fill (arc_segments 32) (thermal_gap 0.508) (thermal_bridge_width 0.508))
+    (polygon
+      (pts
+        (xy 119.253 109.728) (xy 109.728 109.728) (xy 109.728 109.474) (xy 119.253 109.474)
+      )
+    )
+  )
+  (zone (net 0) (net_name "") (layer B.Cu) (hatch edge 0.508)
+    (connect_pads (clearance 0.254))
+    (min_thickness 0.254)
+    (keepout (tracks not_allowed) (vias not_allowed) (copperpour not_allowed))
+    (fill (arc_segments 32) (thermal_gap 0.508) (thermal_bridge_width 0.508))
+    (polygon
+      (pts
+        (xy 164.625257 101.981) (xy 152.4 101.981) (xy 152.4 101.727) (xy 164.625257 101.727)
+      )
+    )
