File: IR-Digipot/Hardware/IR Digipot.kicad_pcb (KiCad board)
At the start: 2 copper layers, 54.9 x 58.4 mm, 133 parts, among them J1 Conn_1x06_Generic, J2 Conn_1x03_Generic, J3 STX-3500-5NTR, J4 STX-3500-5NTR, J5 Molex_1054500101, Q1 MMBT3904, Q2 MMBT3906, Q3 MMBT3904, Q4 MMBT3906, Q5 STL6P3LLH6, Q6 STL6P3LLH6, Q7 STL6P3LLH6, U1 TCM809, U2 PIC18F2550T-I/SO, U3 TSOP754, U4 OPA2134, U5 OPA2134, U6 AD5262, U7 STUSB4500QTR, U8 L7985TR, U9 LM27761, X1 20 MHz

Commit message: Refactor library
Split it into smaller files, which contains components related to each
other.

The goal is to make the library reusable across projects.

The resistors and capacitors are still only generic symbols in the
library and it is still up to designer to link to DigiKey. With time
those components will become accessible via library as well.
Parts:
- C1, C10, C11, C12, C13, C14, C15, C16, C19, C2, C20, C23, C24, C25, C3, C31, C34, C35, C36, C37, C38, C39, C4, C43, C45, C47, C49, C5, C6, C9: footprint Librray:C_0402_1005Metric -> Capacitor_Ceramic:C_0402_1005Metric
- C17, C18: footprint Librray:CP_Elec_8x10 -> Capacitor_Electrolytic:CP_Elec_8x10
- C21, C22, C40, C41, C42, C44, C48: footprint Librray:C_0805_2012Metric -> Capacitor_Ceramic:C_0805_2012Metric
- C26: footprint Librray:C_1206_3216Metric -> Capacitor_Ceramic:C_1206_3216Metric
- C27, C28, C29, C30, C33, C46: footprint Librray:C_0603_1608Metric -> Capacitor_Ceramic:C_0603_1608Metric
- C32: footprint Librray:C_1210_3225Metric -> Capacitor_Ceramic:C_1210_3225Metric
- C7, C8: footprint Librray:CP_Elec_5x5.4 -> Capacitor_Electrolytic:CP_Elec_5x5.4
- D1, D2: footprint Librray:HSMx-C170 -> LED:HSMx-C170
- D10: footprint Librray:D_0603_1610Metric -> Diode:D_0603_1610Metric
- D3, D4, D7: footprint Librray:SOD-523 -> Diode:SOD-523
- D5, D8: footprint Librray:UDFN-2 -> Package_DFN_QFN:UDFN-2
- D6: footprint Librray:SOT-323 -> Package_TO_SOT:SOT-323
- D9: footprint Librray:SOD-323HE -> Diode:SOD-323HE
- FB1, FB2, FB3, FB4: value Ferrite_Bead -> BLM15PG100SN1D; footprint Librray:L_0402_1005Metric -> Inductor:L_0402_1005Metric
- J1: footprint Librray:Conn_1x06_D0.65mm_Pitch2.54mm_staggered -> Connector_Generic:Conn_1x06_D0.65mm_Pitch2.54mm_staggered
- J2: footprint Librray:Conn_1x03_D0.65mm_Pitch2.54mm_staggered -> Connector_Generic:Conn_1x03_D0.65mm_Pitch2.54mm_staggered
- J3, J4: footprint Librray:STX-3500-5NTR -> Connector_Audio:STX-3500-5NTR
- J5: value Molex_1054500101 -> 1054500101; footprint Librray:Molex_1054500101 -> Connector_Data:1054500101
- L1, L3: value ACP3225 -> ACP3225-102-2P-T000; footprint Librray:ACP3225 -> Inductor:ACP3225
- L2: value 22uH -> LQH44PN220MP0L; footprint Librray:L_1515_4040Metric -> Inductor:L_1515_4040Metric
- Q1, Q3: value MMBT3904 -> MMBT3904LT1G; footprint Librray:SOT-23 -> Package_TO_SOT:SOT-23
- Q2, Q4: value MMBT3906 -> MMBT3906LT1G; footprint Librray:SOT-23 -> Package_TO_SOT:SOT-23
- Q5, Q6, Q7: footprint Librray:8-PowerVDFN -> Package_DFN_QFN:8-PowerVDFN
- R1, R10, R11, R12, R13, R14, R15, R16, R17, R18, R19, R2, R20, R21, R22, R23, R24, R25, R26, R27, R28, R29, R3, R30, R31, R32, R33, R34, R35, R36, R37, R38, R39, R4, R40, R41, R42, R43, R44, R45, R5, R6, R7, R8, R9: footprint Librray:R_0402_1005Metric -> Resistor:R_0402_1005Metric
- U1: value TCM809 -> TCM809LVNB713; footprint Librray:SOT-23 -> Package_TO_SOT:SOT-23
- U2: value PIC18F2550T-I/SO -> PIC18F2550T-ISO; footprint Librray:SOIC-28_Width7.50mm_Pitch1.27mm -> Package_SO:SOIC-28_Width7.50mm_Pitch1.27mm
- U3: value TSOP754 -> TSOP75438TR; footprint Librray:TSOP754 -> Interface_Optical:TSOP754
- U4, U5: value OPA2134 -> OPA2134UA_2K5; footprint Librray:SOIC-8_Width3.9mm_Pitch1.27mm -> Package_SO:SOIC-8_Width3.9mm_Pitch1.27mm
- U6: value AD5262 -> AD5262BRUZ50-RL7; footprint Librray:TSSOP-16_4.4x5mm_P0.65mm -> Package_SO:TSSOP-16_4.4x5mm_P0.65mm
- U7: footprint Librray:QFN-24-1EP_4x4mm_P0.5mm_EP2.7x2.7mm -> Package_DFN_QFN:QFN-24-1EP_4x4mm_P0.5mm_EP2.7x2.7mm
- U8: footprint Librray:VFDFPN-10_EP_3x3mm_P0.5mm -> Package_DFN_QFN:VFDFPN-10_EP_3x3mm_P0.5mm
- U9: value LM27761 -> LM27761DSGR; footprint Librray:WSON-8-EP_P0.5mm -> Package_SON:WSON-8-EP_P0.5mm
- X1: value 20 MHz -> ABM8W-20.0000MHZ-4-K1Z-T3; footprint Librray:Crystal_SMD_4Pin_3.2x2.5mm -> Crystal:Crystal_SMD_4Pin_3.2x2.5mm
