File: IR-Digipot/Hardware/Audio.sch (KiCad schematic (older format))
At the start: 46 parts, among them J3 STX-3500-5NTR, J4 STX-3500-5NTR, Q1 MMBT3904, Q2 MMBT3906, Q3 MMBT3904, Q4 MMBT3906, U4 AD5262, U5 OPA2134, U6 OPA2134

Commit message: Continue routing digipot receiver
Minor touches to the USB-C PD tracks, routed signal paths of
audio circuits.

Added missing reset circuits for the digipot.
Parts:
- added C49: 0.1uF, Librray:C_0402_1005Metric, symbol Library:C
- added R42: 3.3K, Librray:R_0402_1005Metric, symbol Library:R
- Q1, Q3: symbol IR-Digipot-rescue:NPN_BEC-Library -> IR-Digipot-rescue:NPN_BEC-Library-IR-Digipot-rescue
- Q2, Q4: symbol IR-Digipot-rescue:PNP_BEC-Library -> IR-Digipot-rescue:PNP_BEC-Library-IR-Digipot-rescue
Connections:
- wire segments 175 -> 188

Commit message: Remove connection from audio jacks switches
Were wrongly connected to ground. The idea was to connect
unused pads to big copper mass to give mechanical rigidity.

Should be done using non-connected net.
Connections:
- net GNDA: no longer J3.4, J3.5, J4.4, J4.5
Changed lines of the file:
@@
 	1    0    0    1
 $EndComp
-Wire Wire Line
-	9200 4450 9100 4450
-Wire Wire Line
-	9100 4450 9100 4550
-Wire Wire Line
-	9200 4550 9100 4550
-Connection ~ 9100 4550
-Wire Wire Line
-	9100 4550 9100 4850
 $Comp
 L Library:R R?
@@
 Wire Wire Line
 	7350 3500 7350 3550
-$Comp
-L power:GNDA #PWR0131
-U 1 1 5FF0BD63
-P 9100 4850
-F 0 "#PWR0131" H 9100 4600 50  0001 C CNN
-F 1 "GNDA" H 9105 4677 50  0000 C CNN
-F 2 "" H 9100 4850 50  0001 C CNN
-F 3 "" H 9100 4850 50  0001 C CNN
-	1    9100 4850
-	1    0    0    -1
-$EndComp
-$Comp
-L power:GNDA #PWR?
-U 1 1 600230ED
-P 9100 6000
-F 0 "#PWR?" H 9100 5750 50  0001 C CNN
-F 1 "GNDA" H 9105 5827 50  0000 C CNN
-F 2 "" H 9100 6000 50  0001 C CNN
-F 3 "" H 9100 6000 50  0001 C CNN
-	1    9100 6000
-	1    0    0    -1
-$EndComp
-Wire Wire Line
-	9100 6000 9100 5700
-Wire Wire Line
-	9100 5600 9150 5600
-Wire Wire Line
-	9150 5700 9100 5700
-Connection ~ 9100 5700
-Wire Wire Line
-	9100 5700 9100 5600
 $EndSCHEMATC

Commit message: Prevision digipot power from +5VD
The idea is to try to bring digipot running before powering on
buffers with the goal of programming proper volume on power on.

Should help reducing popping on power on.
Parts:
- added R?: NC, Librray:R_0402_1005Metric, symbol Library:R
Connections:
- net +5VA: no longer R42.1
- net DIGIPOT_VL: now reaches FB1.2, U4.13 (VL)
- net DIGIPOT_VL: now also R42.1, R?.1
- new net +5VD: R?.2
Other:
- moved on the sheet: R42
Changed lines of the file:
@@
 Wire Wire Line
 	8950 3300 8950 3350
-Wire Wire Line
-	8950 1600 8950 1850
 $Comp
 L Library:Ferrite_Bead FB1
@@
 L power:+5VA #PWR0110
 U 1 1 5FE3C7B2
-P 8950 1600
-F 0 "#PWR0110" H 8950 1450 50  0001 C CNN
-F 1 "+5VA" H 8965 1773 50  0000 C CNN
-F 2 "" H 8950 1600 50  0001 C CNN
-F 3 "" H 8950 1600 50  0001 C CNN
-	1    8950 1600
-	1    0    0    -1
-$EndComp
-$Comp
-L power:+5VA #PWR063
-U 1 1 5FF77FA3
-P 7350 2250
-F 0 "#PWR063" H 7350 2100 50  0001 C CNN
-F 1 "+5VA" H 7365 2423 50  0000 C CNN
-F 2 "" H 7350 2250 50  0001 C CNN
-F 3 "" H 7350 2250 50  0001 C CNN
-	1    7350 2250
+P 8950 1450
+F 0 "#PWR0110" H 8950 1300 50  0001 C CNN
+F 1 "+5VA" H 8965 1623 50  0000 C CNN
+F 2 "" H 8950 1450 50  0001 C CNN
+F 3 "" H 8950 1450 50  0001 C CNN
+	1    8950 1450
 	1    0    0    -1
 $EndComp
@@
 L Library:R R?
 U 1 1 5FF44F9D
-P 7450 2450
+P 7150 2350
 AR Path="/5FE20DA8/5FF44F9D" Ref="R?"  Part="1"
 AR Path="/5FE379B8/5FF44F9D" Ref="R42"  Part="1"
-F 0 "R42" H 7450 2450 50  0000 L BNN
-F 1 "3.3K" H 7450 2350 50  0000 L BNN
-F 2 "Librray:R_0402_1005Metric" H 7450 2450 50  0001 C CNN
-F 3 "" H 7450 2450 50  0001 C CNN
-F 4 "CRGCQ 0402 3K3 1%" H 7450 2450 50  0001 C CNN "Description"
-F 5 "TE Connectivity Passive Product" H 7450 2450 50  0001 C CNN "Manufacturer"
-F 6 "CRGCQ0402F3K3" H 7450 2450 50  0001 C CNN "Manufacturer Part Number"
-F 7 "A129633CT-ND" H 7450 2450 50  0001 C CNN "Digi-Key Part Number"
-	1    7450 2450
-	1    0    0    -1
+F 0 "R42" V 7150 2400 50  0000 L BNN
+F 1 "3.3K" V 7150 2100 50  0000 L BNN
+F 2 "Librray:R_0402_1005Metric" H 7150 2350 50  0001 C CNN
+F 3 "" H 7150 2350 50  0001 C CNN
+F 4 "CRGCQ 0402 3K3 1%" H 7150 2350 50  0001 C CNN "Description"
+F 5 "TE Connectivity Passive Product" H 7150 2350 50  0001 C CNN "Manufacturer"
+F 6 "CRGCQ0402F3K3" H 7150 2350 50  0001 C CNN "Manufacturer Part Number"
+F 7 "A129633CT-ND" H 7150 2350 50  0001 C CNN "Digi-Key Part Number"
+	1    7150 2350
+	0    -1   -1   0
 $EndComp
 Wire Wire Line
@@
 Wire Wire Line
 	7050 3100 8500 3100
-Wire Wire Line
-	7350 2250 7350 2300
-Wire Wire Line
-	7350 2600 7350 2750
 Wire Wire Line
 	8500 2750 7350 2750
@@
 Wire Wire Line
 	7350 3500 7350 3550
+Connection ~ 9250 1850
+$Comp
+L Library:R R?
+U 1 1 6004A6D1
+P 9550 1650
+AR Path="/5FE20DA8/6004A6D1" Ref="R?"  Part="1"
+AR Path="/5FE379B8/6004A6D1" Ref="R?"  Part="1"
+AR Path="/5FF173B2/6004A6D1" Ref="R?"  Part="1"
+AR Path="/5FF86B45/6004A6D1" Ref="R?"  Part="1"
+F 0 "R?" V 9550 1700 50  0000 L BNN
+F 1 "NC" V 9550 1500 50  0000 L BNN
+F 2 "Librray:R_0402_1005Metric" H 9550 1650 50  0001 C CNN
+F 3 "" H 9550 1650 50  0001 C CNN
+	1    9550 1650
+	-1   0    0    1
+$EndComp
+Wire Wire Line
+	8950 1450 8950 1850
+Wire Wire Line
+	9650 1850 9650 1800
+Wire Wire Line
+	9250 1850 9650 1850
+$Comp
+L power:+5VD #PWR?
+U 1 1 60067AD0
+P 9650 1450
+F 0 "#PWR?" H 9650 1300 50  0001 C CNN
+F 1 "+5VD" H 9665 1623 50  0000 C CNN
+F 2 "" H 9650 1450 50  0001 C CNN
+F 3 "" H 9650 1450 50  0001 C CNN
+	1    9650 1450
+	1    0    0    -1
+$EndComp
+Wire Wire Line
+	9650 1450 9650 1500
+Wire Wire Line
+	9650 1850 10500 1850
+Connection ~ 9650 1850
+Text Label 10500 1850 2    50   ~ 0
+DIGIPOT_VL
+Text Label 6450 2450 0    50   ~ 0
+DIGIPOT_VL
+Wire Wire Line
+	7300 2450 7350 2450
+Wire Wire Line
+	7350 2450 7350 2750
+Wire Wire Line
+	6450 2450 7000 2450
 $EndSCHEMATC
