File: IR-Digipot/Hardware/Audio.sch (KiCad schematic (older format))
At the start: 49 parts, among them J3 STX-3500-5NTR, J4 STX-3500-5NTR, Q1 MMBT3904, Q2 MMBT3906, Q3 MMBT3904, Q4 MMBT3906, U4 AD5262, U5 OPA2134, U6 OPA2134

Commit message: Tweak digipot preamp gain
Allows to feed professional equipment level of signal which is
3.472 Vpp. There is enough swing to do 4 Vpp with the new gain.
Parts:
- R10: renamed from R8; value 3.3K -> 12K; Description CRGCQ 0402 3K3 1% -> CRGCQ 0402 12K 1%; Digi-Key Part Number A129633CT-ND -> A129640CT-ND; Manufacturer Part Number CRGCQ0402F3K3 -> CRGCQ0402F12K
- R13: renamed from R15; value 3.3K -> 12K; Description CRGCQ 0402 3K3 1% -> CRGCQ 0402 12K 1%; Digi-Key Part Number A129633CT-ND -> A129640CT-ND; Manufacturer Part Number CRGCQ0402F3K3 -> CRGCQ0402F12K
- R14: renamed from R16; value 3.3K -> 12K; Description CRGCQ 0402 3K3 1% -> CRGCQ 0402 12K 1%; Digi-Key Part Number A129633CT-ND -> A129640CT-ND; Manufacturer Part Number CRGCQ0402F3K3 -> CRGCQ0402F12K
- R17: renamed from R11; value 33K -> 22K; Description CRGCQ 0402 33K 1% -> CRGCQ 0402 22K 1%; Digi-Key Part Number A129645CT-ND -> A129643CT-ND; Manufacturer Part Number CRGCQ0402F33K -> CRGCQ0402F22K
- R18: renamed from R12; value 33K -> 22K; Description CRGCQ 0402 33K 1% -> CRGCQ 0402 22K 1%; Digi-Key Part Number A129645CT-ND -> A129643CT-ND; Manufacturer Part Number CRGCQ0402F33K -> CRGCQ0402F22K
- R7: renamed from R13; value 33K -> 22K; Description CRGCQ 0402 33K 1% -> CRGCQ 0402 22K 1%; Digi-Key Part Number A129645CT-ND -> A129643CT-ND; Manufacturer Part Number CRGCQ0402F33K -> CRGCQ0402F22K
- R8: renamed from R14; value 33K -> 22K; Description CRGCQ 0402 33K 1% -> CRGCQ 0402 22K 1%; Digi-Key Part Number A129645CT-ND -> A129643CT-ND; Manufacturer Part Number CRGCQ0402F33K -> CRGCQ0402F22K
- R9: renamed from R7; value 3.3K -> 12K; Description CRGCQ 0402 3K3 1% -> CRGCQ 0402 12K 1%; Digi-Key Part Number A129633CT-ND -> A129640CT-ND; Manufacturer Part Number CRGCQ0402F3K3 -> CRGCQ0402F12K
- renumbered C17 to C11, C18 to C12, C11 to C13, C12 to C14, C23 to C15, C24 to C16, C21 to C17, C22 to C18, C15 to C19, C16 to C20, C5 to C21, C6 to C22, C49 to C23, C7 to C24, C8 to C25, C19 to C5, C20 to C6, C13 to C7, C14 to C8, R9 to R11, R10 to R12, R17 to R15, R18 to R16, R42 to R19, R43 to R20, U6 to U4, U4 to U6
Other:
- moved on the sheet: J4

Commit message: Add status LEDs to the digipot
Parts:
- renumbered D1 to D3, D2 to D4, R8 to R10, R9 to R11, R10 to R12, R11 to R13, R12 to R14, R13 to R15, R14 to R16, R15 to R17, R16 to R18, R17 to R19, R18 to R20, R19 to R21, R20 to R22, R5 to R7, R6 to R8, R7 to R9

Commit message: Refactor library
Split it into smaller files, which contains components related to each
other.

The goal is to make the library reusable across projects.

The resistors and capacitors are still only generic symbols in the
library and it is still up to designer to link to DigiKey. With time
those components will become accessible via library as well.
Parts:
- C10, C11, C12, C13, C14, C15, C16, C19, C20, C23, C24, C25, C5, C6, C9: footprint Librray:C_0402_1005Metric -> Capacitor_Ceramic:C_0402_1005Metric; symbol Library:C -> Capacitor_Ceramic:C
- C17, C18: footprint Librray:CP_Elec_8x10 -> Capacitor_Electrolytic:CP_Elec_8x10; symbol Library:CP -> Capacitor_Electrolytic:CP
- C21, C22: footprint Librray:C_0805_2012Metric -> Capacitor_Ceramic:C_0805_2012Metric; symbol Library:C -> Capacitor_Ceramic:C
- C7, C8: footprint Librray:CP_Elec_5x5.4 -> Capacitor_Electrolytic:CP_Elec_5x5.4; symbol Library:CP -> Capacitor_Electrolytic:CP
- D3, D4: footprint Librray:SOD-523 -> Diode:SOD-523; symbol Library:D -> Diode:D
- FB1: value Ferrite_Bead -> BLM15PG100SN1D; footprint Librray:L_0402_1005Metric -> Inductor:L_0402_1005Metric; symbol Library:Ferrite_Bead -> Inductor:BLM15PG100SN1D; Detailed Description (none) -> 10 Ohms @ 100MHz 1 Power Line Ferrite Bead 0402 (1005 Metri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
- J3, J4: footprint Librray:STX-3500-5NTR -> Connector_Audio:STX-3500-5NTR; symbol Library:STX-3500-5NTR -> Connector_Audio:STX-3500-5NTR; Detailed Description (none) -> 3.50mm (0.141\", 1/8\", Mini Plug) - Headphone Phone Jack S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
- Q1, Q3: value MMBT3904 -> MMBT3904LT1G; footprint Librray:SOT-23 -> Package_TO_SOT:SOT-23; symbol IR-Digipot-rescue:NPN_BEC-Library-IR-Digipot-rescue -> Transistor_BJT:MMBT3904LT1G; Base Part Number (none) -> MMBT3904; Detailed Description (none) -> Bipolar (BJT) Transistor NPN 40V 200mA 300MHz 300mW Surface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
- Q2, Q4: value MMBT3906 -> MMBT3906LT1G; footprint Librray:SOT-23 -> Package_TO_SOT:SOT-23; symbol IR-Digipot-rescue:PNP_BEC-Library-IR-Digipot-rescue -> Transistor_BJT:MMBT3906LT1G; Base Part Number (none) -> MMBT3906; Detailed Description (none) -> Bipolar (BJT) Transistor PNP 40V 200mA 250MHz 300mW Surface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
- R10, R11, R12, R13, R14, R15, R16, R17, R18, R19, R20, R21, R22, R7, R8, R9: footprint Librray:R_0402_1005Metric -> Resistor:R_0402_1005Metric; symbol Library:R -> Resistor:R
- U4, U5: value OPA2134 -> OPA2134UA_2K5; footprint Librray:SOIC-8_Width3.9mm_Pitch1.27mm -> Package_SO:SOIC-8_Width3.9mm_Pitch1.27mm; symbol Library:OPA2134 -> Amplifier_Operational:OPA2134UA_2K5; Detailed Description (none) -> Audio Amplifier 2 Circuit 8-SOIC
- U4, U5: value OPA2134 -> OPA2134UA_2K5; footprint Librray:SOIC-8_Width3.9mm_Pitch1.27mm -> Package_SO:SOIC-8_Width3.9mm_Pitch1.27mm; symbol Library:OPA2134 -> Amplifier_Operational:OPA2134UA_2K5; Description (none) -> IC AUDIO 2 CIRCUIT 8SOIC; Detailed Description (none) -> Audio Amplifier 2 Circuit 8-SOIC; Digi-Key Part Number (none) -> 296-22024-1-ND; Manufacturer (none) -> Texas Instruments; Manufacturer Part Number (none) -> OPA2134UA/2K5
- U4, U5: value OPA2134 -> OPA2134UA_2K5; footprint Librray:SOIC-8_Width3.9mm_Pitch1.27mm -> Package_SO:SOIC-8_Width3.9mm_Pitch1.27mm; symbol Library:OPA2134 -> Amplifier_Operational:OPA2134UA_2K5
- U6: value AD5262 -> AD5262BRUZ50-RL7; footprint Librray:TSSOP-16_4.4x5mm_P0.65mm -> Package_SO:TSSOP-16_4.4x5mm_P0.65mm; symbol Library:AD5262 -> Potentiometer_Digital:AD5262BRUZ50-RL7; Detailed Description (none) -> Digital Potentiometer 50k Ohm 2 Circuit 256 Taps SPI Interf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
