File: IR-Digipot/Hardware/CPU.sch (KiCad schematic (older format))
At the start: 18 parts, among them J1 Conn_1x06_Generic, J2 Conn_1x03_Generic, U1 TCM809, U2 PIC18F2550T-I/SO, U3 TSOP754, X1 20 MHz

Commit message: Refactor library
Split it into smaller files, which contains components related to each
other.

The goal is to make the library reusable across projects.

The resistors and capacitors are still only generic symbols in the
library and it is still up to designer to link to DigiKey. With time
those components will become accessible via library as well.
Parts:
- C1, C2, C3, C4: footprint Librray:C_0402_1005Metric -> Capacitor_Ceramic:C_0402_1005Metric; symbol Library:C -> Capacitor_Ceramic:C
- D1, D2: footprint Librray:HSMx-C170 -> LED:HSMx-C170; symbol Library:LED -> LED:HSMG-C170; Detailed Description (none) -> Green 572nm LED Indication - Discrete 2.2V 0805 (2012 Metri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
- J1: footprint Librray:Conn_1x06_D0.65mm_Pitch2.54mm_staggered -> Connector_Generic:Conn_1x06_D0.65mm_Pitch2.54mm_staggered; symbol Library:Conn_1x06_Generic -> Connector_Generic:Conn_1x06_Generic
- J2: footprint Librray:Conn_1x03_D0.65mm_Pitch2.54mm_staggered -> Connector_Generic:Conn_1x03_D0.65mm_Pitch2.54mm_staggered; symbol Library:Conn_1x03_Generic -> Connector_Generic:Conn_1x03_Generic
- R1, R2, R3, R4, R5, R6: footprint Librray:R_0402_1005Metric -> Resistor:R_0402_1005Metric; symbol Library:R -> Resistor:R
- U1: value TCM809 -> TCM809LVNB713; footprint Librray:SOT-23 -> Package_TO_SOT:SOT-23; symbol Library:TCM809 -> Power_Supervisor:TCM809LVNB713; Detailed Description (none) -> Supervisor Push-Pull, Totem Pole 1 Channel SOT-23-3
- U2: value PIC18F2550T-I/SO -> PIC18F2550T-ISO; footprint Librray:SOIC-28_Width7.50mm_Pitch1.27mm -> Package_SO:SOIC-28_Width7.50mm_Pitch1.27mm; symbol Library:PIC18F2550 -> Microcontroller:PIC18F2550T-ISO; Detailed Description (none) -> PIC PIC® 18F Microcontroller IC 8-Bit 48MHz 32KB (16K x 16)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; Digi-Key Part Number PIC18F2550T-I/SOCT-ND -> PIC18LF2550-I/SO-ND; Manufacturer Part Number PIC18F2550T-I/SO -> PIC18LF2550-I/SO
- U3: value TSOP754 -> TSOP75438TR; footprint Librray:TSOP754 -> Interface_Optical:TSOP754; symbol Library:TSOP754 -> Interface_Optical:TSOP75438TR; Detailed Description (none) -> Remote Receiver Sensor, 38.0kHz 45m Surface Mount
- X1: value 20 MHz -> ABM8W-20.0000MHZ-4-K1Z-T3; footprint Librray:Crystal_SMD_4Pin_3.2x2.5mm -> Crystal:Crystal_SMD_4Pin_3.2x2.5mm; symbol Library:Crystal_GND24 -> Crystal:ABM8W-20.0000MHZ-4-K1Z-T3; Detailed Description (none) -> 20MHz ±10ppm Crystal 4pF 50 Ohms 4-SMD, No Lead; Frequency (none) -> 20MHz
