File: IR-Digipot/Hardware/Power Delivery.sch (KiCad schematic (older format))
At the start: 26 parts, among them J5 Molex_1054500101, Q5 STL6P3LLH6, Q6 STL6P3LLH6, U7 STUSB4500QTR

Commit message: Wire high-side switch FET for +5VA
The PIC port should be able to draw enough current to
properly control the switch.
Parts:
- U7: symbol Library:STUSB4500QTR -> IR-Digipot-rescue:STUSB4500QTR-Library
Changed lines of the file:
@@
 	3600 3150 2100 3150
 $Comp
-L Library:STUSB4500QTR U7
+L IR-Digipot-rescue:STUSB4500QTR-Library U7
 U 1 1 5FE5C56B
 P 6900 4450

Commit message: Continue routing digipot receiver
Minor touches to the USB-C PD tracks, routed signal paths of
audio circuits.

Added missing reset circuits for the digipot.
Parts:
- U7: symbol IR-Digipot-rescue:STUSB4500QTR-Library -> IR-Digipot-rescue:STUSB4500QTR-Library-IR-Digipot-rescue
Changed lines of the file:
@@
 	3600 3150 2100 3150
 $Comp
-L IR-Digipot-rescue:STUSB4500QTR-Library U7
+L IR-Digipot-rescue:STUSB4500QTR-Library-IR-Digipot-rescue U7
 U 1 1 5FE5C56B
 P 6900 4450
+AR Path="/5FE5C56B" Ref="U7"  Part="1"
+AR Path="/5FF173B2/5FE5C56B" Ref="U7"  Part="1"
 F 0 "U7" H 7200 5250 50  0000 L BNN
 F 1 "STUSB4500QTR" H 7200 5150 50  0000 L BNN

Commit message: Tweak digipot preamp gain
Allows to feed professional equipment level of signal which is
3.472 Vpp. There is enough swing to do 4 Vpp with the new gain.
Parts:
- renumbered C25 to C26, C29 to C27, C26 to C28, C27 to C29, C28 to C30, C30 to C31, R19 to R21, R20 to R22, R21 to R23, R22 to R26, R26 to R27, R30 to R28, R27 to R29, R23 to R30, R28 to R31, R29 to R32

Commit message: Add status LEDs to the digipot
Parts:
- renumbered D3 to D5, D4 to D6, D5 to D7, D6 to D8, R21 to R23, R22 to R24, R23 to R25, R24 to R26, R25 to R27, R26 to R28, R27 to R29, R28 to R30, R29 to R31, R30 to R32, R31 to R33, R32 to R34

Commit message: Refactor library
Split it into smaller files, which contains components related to each
other.

The goal is to make the library reusable across projects.

The resistors and capacitors are still only generic symbols in the
library and it is still up to designer to link to DigiKey. With time
those components will become accessible via library as well.
Parts:
- C26: footprint Librray:C_1206_3216Metric -> Capacitor_Ceramic:C_1206_3216Metric; symbol Library:C -> Capacitor_Ceramic:C
- C27, C28, C29, C30: footprint Librray:C_0603_1608Metric -> Capacitor_Ceramic:C_0603_1608Metric; symbol Library:C -> Capacitor_Ceramic:C
- C31: footprint Librray:C_0402_1005Metric -> Capacitor_Ceramic:C_0402_1005Metric; symbol Library:C -> Capacitor_Ceramic:C
- D5, D8: footprint Librray:UDFN-2 -> Package_DFN_QFN:UDFN-2; symbol Library:D_ZENNER -> Diode:D_ZENNER
- D6: footprint Librray:SOT-323 -> Package_TO_SOT:SOT-323; symbol Library:D_ZENNER_DUAL_CATHODE -> Diode:D_ZENNER_DUAL_CATHODE
- D7: footprint Librray:SOD-523 -> Diode:SOD-523; symbol Library:D_SCHOTTKY -> Diode:D_SCHOTTKY
- J5: value Molex_1054500101 -> 1054500101; footprint Librray:Molex_1054500101 -> Connector_Data:1054500101; symbol Library:Molex_1054500101 -> Connector_Data:1054500101; Detailed Description (none) -> USB-C (USB TYPE-C) USB 3.2 Gen 2 (USB 3.1 Gen 2, Superspeed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; Drawing (none) -> https://www.molex.com/pdm_docs/sd/1054500101_sd.pdf
- Q5, Q6: footprint Librray:8-PowerVDFN -> Package_DFN_QFN:8-PowerVDFN; symbol Library:P-CHANNEL-SGD -> Transistor_FET:STL6P3LLH6; Detailed Description (none) -> P-Channel 30V 6A (Tc) 2.9W (Tc) Surface Mount PowerFlat™ (3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
- R23, R24, R25, R26, R27, R28, R29, R30, R31, R32, R33, R34: footprint Librray:R_0402_1005Metric -> Resistor:R_0402_1005Metric; symbol Library:R -> Resistor:R
- U7: footprint Librray:QFN-24-1EP_4x4mm_P0.5mm_EP2.7x2.7mm -> Package_DFN_QFN:QFN-24-1EP_4x4mm_P0.5mm_EP2.7x2.7mm; symbol IR-Digipot-rescue:STUSB4500QTR-Library-IR-Digipot-rescue -> Interface_USB:STUSB4500QTR; Detailed Description (none) -> USB Controller USB 2.0 I²C Interface 24-QFN (4x4)
