File: IR-Controller/Hardware/IR-Controller.kicad_pcb (KiCad board)
At the start: 2 copper layers, 1 part, among them U1 PIC18LF2550

Commit message: Controller: Add battery holder
Parts:
- added BT1: Battery, Librray:BC-2003, B.Cu at (82.5, 120.7)
- moved U1 8.77 mm to (82.5, 95.2)
Changed lines of the file:
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@@
     (tracks 0)
     (zones 0)
-    (modules 1)
+    (modules 2)
     (nets 28)
   )
@@
     (pad_to_mask_clearance 0)
     (aux_axis_origin 0 0)
-    (visible_elements FFFFFF7F)
+    (visible_elements 7FFFFFFF)
     (pcbplotparams
       (layerselection 0x010fc_ffffffff)
@@
     (add_net "Net-(U1-Pad9)")
   )
+  (module Librray:BC-2003 (layer B.Cu)
+    (at 82.55 120.65)
+    (fp_text reference BT1 (at 0 4.445) (layer B.SilkS)
+      (effects (font (size 1 1) (thickness 0.15)) (justify mirror))
+    )
+    (fp_text value Battery (at 0 -3.556) (layer B.Fab)
+      (effects (font (size 1 1) (thickness 0.15)) (justify mirror))
+    )
+    (fp_arc (start 0 0) (end -9.524998 -2.920998) (angle 145.9019419) (layer B.CrtYd) (width 0.12))
+    (fp_arc (start 0 0) (end 9.524999 2.920999) (angle 145.9019381) (layer B.CrtYd) (width 0.12))
+    (fp_circle (center 0 0) (end 10 0) (layer B.Fab) (width 0.12))
+    (fp_line (start -13.335 -2.921) (end -13.335 2.921) (layer B.CrtYd) (width 0.12))
+    (fp_line (start 13.335 -2.921) (end 13.335 2.921) (layer B.CrtYd) (width 0.12))
+    (fp_line (start -13.335 2.921) (end -9.524999 2.921) (layer B.CrtYd) (width 0.12))
+    (fp_line (start -13.335 -2.921) (end -9.524999 -2.920999) (layer B.CrtYd) (width 0.12))
+    (fp_line (start 13.335 2.921) (end 9.524999 2.920999) (layer B.CrtYd) (width 0.12))
+    (fp_line (start 13.335 -2.921) (end 9.524997 -2.921) (layer B.CrtYd) (width 0.12))
+    (pad 1 smd rect (at 11.905 0) (size 2.6 5.56) (layers B.Cu B.Paste B.Mask)
+      (net 12 +3V0))
+    (pad 2 smd rect (at 0 0) (size 8.34 5.56) (layers B.Cu B.Paste B.Mask)
+      (net 10 GND))
+    (pad 1 smd rect (at -11.905 0) (size 2.6 5.56) (layers B.Cu B.Paste B.Mask)
+      (net 12 +3V0))
+    (model ${KIPRJMOD}/../../Library/Models/BC-2003/BC-2003.wrl
+      (at (xyz 0 0 0))
+      (scale (xyz 0.3937007874015748 0.3937007874015748 0.3937007874015748))
+      (rotate (xyz 0 0 0))
+    )
+  )
   (module Librray:SOIC-28_Width7.50mm_Pitch1.27mm (layer B.Cu)
-    (at 89.662 100.3808 180)
+    (at 82.55 95.25 180)
     (attr smd)
     (fp_text reference U1 (at 0 10.005) (layer B.SilkS)
@@
       (effects (font (size 1 1) (thickness 0.15)) (justify mirror))
     )
+    (fp_line (start 3.175 8.255) (end 3.175 -8.255) (layer B.SilkS) (width 0.12))
+    (fp_line (start 3.175 -8.255) (end -3.175 -8.255) (layer B.SilkS) (width 0.12))
+    (fp_line (start -3.175 -8.255) (end -3.175 7.62) (layer B.SilkS) (width 0.12))
+    (fp_line (start 5.65 8.76) (end 5.65 -8.76) (layer B.CrtYd) (width 0.05))
+    (fp_line (start 5.65 -8.76) (end -5.65 -8.76) (layer B.CrtYd) (width 0.05))
+    (fp_line (start -5.65 -8.76) (end -5.65 8.76) (layer B.CrtYd) (width 0.05))
+    (fp_line (start -5.65 8.76) (end 5.65 8.76) (layer B.CrtYd) (width 0.05))
+    (fp_line (start -2.54 8.255) (end -3.175 7.62) (layer B.SilkS) (width 0.12))
+    (fp_line (start 3.175 8.255) (end -2.54 8.255) (layer B.SilkS) (width 0.12))
+    (fp_circle (center -1.905 6.985) (end -1.905 6.6675) (layer B.SilkS) (width 0.12))
     (fp_circle (center -4.572 9.271) (end -4.572 9.144) (layer B.SilkS) (width 0.254))
-    (fp_circle (center -1.905 6.985) (end -1.905 6.6675) (layer B.SilkS) (width 0.12))
-    (fp_line (start 3.175 8.255) (end -2.54 8.255) (layer B.SilkS) (width 0.12))
-    (fp_line (start -2.54 8.255) (end -3.175 7.62) (layer B.SilkS) (width 0.12))
-    (fp_line (start -5.65 8.76) (end 5.65 8.76) (layer B.CrtYd) (width 0.05))
-    (fp_line (start -5.65 -8.76) (end -5.65 8.76) (layer B.CrtYd) (width 0.05))
-    (fp_line (start 5.65 -8.76) (end -5.65 -8.76) (layer B.CrtYd) (width 0.05))
-    (fp_line (start 5.65 8.76) (end 5.65 -8.76) (layer B.CrtYd) (width 0.05))
-    (fp_line (start -3.175 -8.255) (end -3.175 7.62) (layer B.SilkS) (width 0.12))
-    (fp_line (start 3.175 -8.255) (end -3.175 -8.255) (layer B.SilkS) (width 0.12))
-    (fp_line (start 3.175 8.255) (end 3.175 -8.255) (layer B.SilkS) (width 0.12))
     (pad 14 smd rect (at -4.572 -8.255 270) (size 0.5 1.5875) (layers B.Cu B.Paste B.Mask)
       (net 1 "Net-(U1-Pad14)"))

Commit message: Controller: Add IR LED
Parts:
- added C1: 0.1uF, Librray:C_0402_1005Metric, B.Cu at (75.6, 97.8)
- added D1: IN-S126ESGHIR, Librray:IN-S126ESGHIR, B.Cu at (82.5, 80.6)
- BT1: value Battery -> BC-2003
Changed lines of the file:
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@@
     (tracks 0)
     (zones 0)
-    (modules 2)
-    (nets 28)
+    (modules 4)
+    (nets 30)
   )
   (page A4)
@@
     (46 B.CrtYd user)
     (47 F.CrtYd user)
-    (48 B.Fab user)
-    (49 F.Fab user)
+    (48 B.Fab user hide)
+    (49 F.Fab user hide)
   )
   (setup
@@
   (net 26 "Net-(U1-Pad1)")
   (net 27 "Net-(U1-Pad28)")
+  (net 28 "Net-(D1-Pad2)")
+  (net 29 "Net-(D1-Pad1)")
   (net_class Default "This is the default net class."
     (clearance 0.2)
@@
     (add_net +3V0)
     (add_net GND)
+    (add_net "Net-(D1-Pad1)")
+    (add_net "Net-(D1-Pad2)")
     (add_net "Net-(U1-Pad1)")
     (add_net "Net-(U1-Pad10)")
@@
     (add_net "Net-(U1-Pad9)")
   )
+  (module Librray:IN-S126ESGHIR (layer B.Cu)
+    (at 82.55 80.645)
+    (fp_text reference D1 (at 0 1.524) (layer B.SilkS)
+      (effects (font (size 0.6 0.6) (thickness 0.15)) (justify mirror))
+    )
+    (fp_text value IN-S126ESGHIR (at 0 -2.794) (layer B.Fab)
+      (effects (font (size 1 1) (thickness 0.15)) (justify mirror))
+    )
+    (fp_line (start -2.159 -0.762) (end -2.159 0.762) (layer B.SilkS) (width 0.12))
+    (fp_line (start -2.159 -2.032) (end 2.159 -2.032) (layer F.CrtYd) (width 0.12))
+    (fp_line (start 2.159 -2.032) (end 2.159 0.889) (layer F.CrtYd) (width 0.12))
+    (fp_line (start 2.159 0.889) (end -2.159 0.889) (layer F.CrtYd) (width 0.12))
+    (fp_line (start -2.159 0.889) (end -2.159 -2.032) (layer F.CrtYd) (width 0.12))
+    (pad "" smd rect (at 0 0) (size 0.6 1.6) (layers B.Cu B.Paste B.Mask))
+    (pad 2 smd rect (at 1.5 0) (size 1 1.6) (layers B.Cu B.Paste B.Mask)
+      (net 28 "Net-(D1-Pad2)"))
+    (pad 1 smd rect (at -1.5 0) (size 1 1.6) (layers B.Cu B.Paste B.Mask)
+      (net 29 "Net-(D1-Pad1)"))
+    (model ${KIPRJMOD}/../../Library/Models/IN-S126ESGHIR/IN-S126ESGHIR.wrl
+      (at (xyz 0 0 0))
+      (scale (xyz 0.3937007874015748 0.3937007874015748 0.3937007874015748))
+      (rotate (xyz 0 0 0))
+    )
+  )
+  (module Librray:C_0402_1005Metric (layer B.Cu)
+    (at 75.565 97.79 90)
+    (fp_text reference C1 (at 0 -1.27 90) (layer B.SilkS)
+      (effects (font (size 0.6 0.6) (thickness 0.15)) (justify mirror))
+    )
+    (fp_text value 0.1uF (at 0 -1.524 90) (layer B.Fab)
+      (effects (font (size 1 1) (thickness 0.15)) (justify mirror))
+    )
+    (fp_line (start -0.889 -0.381) (end 0.889 -0.381) (layer B.CrtYd) (width 0.12))
+    (fp_line (start -0.889 0.381) (end -0.889 -0.381) (layer B.CrtYd) (width 0.12))
+    (fp_line (start 0.889 0.381) (end -0.889 0.381) (layer B.CrtYd) (width 0.12))
+    (fp_line (start 0.889 -0.381) (end 0.889 0.381) (layer B.CrtYd) (width 0.12))
+    (pad 2 smd rect (at 0.508 0 90) (size 0.6 0.7) (layers B.Cu B.Paste B.Mask)
+      (net 12 +3V0))
+    (pad 1 smd rect (at -0.508 0 90) (size 0.6 0.7) (layers B.Cu B.Paste B.Mask)
+      (net 10 GND))
+    (model ${KISYS3DMOD}/Capacitor_SMD.3dshapes/C_0402_1005Metric.wrl
+      (at (xyz 0 0 0))
+      (scale (xyz 1 1 1))
+      (rotate (xyz 0 0 0))
+    )
+  )
   (module Librray:BC-2003 (layer B.Cu)
     (at 82.55 120.65)
@@
       (effects (font (size 1 1) (thickness 0.15)) (justify mirror))
     )
-    (fp_text value Battery (at 0 -3.556) (layer B.Fab)
-      (effects (font (size 1 1) (thickness 0.15)) (justify mirror))
-    )
-    (fp_arc (start 0 0) (end -9.524998 -2.920998) (angle 145.9019419) (layer B.CrtYd) (width 0.12))
-    (fp_arc (start 0 0) (end 9.524999 2.920999) (angle 145.9019381) (layer B.CrtYd) (width 0.12))
+    (fp_text value BC-2003 (at 0 -3.556) (layer B.Fab)
+      (effects (font (size 1 1) (thickness 0.15)) (justify mirror))
+    )
     (fp_circle (center 0 0) (end 10 0) (layer B.Fab) (width 0.12))
     (fp_line (start -13.335 -2.921) (end -13.335 2.921) (layer B.CrtYd) (width 0.12))
@@
     (fp_line (start 13.335 2.921) (end 9.524999 2.920999) (layer B.CrtYd) (width 0.12))
     (fp_line (start 13.335 -2.921) (end 9.524997 -2.921) (layer B.CrtYd) (width 0.12))
+    (fp_arc (start 0 0) (end -9.524998 -2.920998) (angle 145.9019419) (layer B.CrtYd) (width 0.12))
+    (fp_arc (start 0 0) (end 9.524999 2.920999) (angle 145.9019381) (layer B.CrtYd) (width 0.12))
     (pad 1 smd rect (at 11.905 0) (size 2.6 5.56) (layers B.Cu B.Paste B.Mask)
       (net 12 +3V0))
@@
     (at 82.55 95.25 180)
     (attr smd)
-    (fp_text reference U1 (at 0 10.005) (layer B.SilkS)
-      (effects (font (size 1 1) (thickness 0.15)) (justify mirror))
+    (fp_text reference U1 (at 0 9.525) (layer B.SilkS)
+      (effects (font (size 0.6 0.6) (thickness 0.15)) (justify mirror))
     )
     (fp_text value PIC18LF2550 (at 0 0 90) (layer B.Fab)

Commit message: Controller: Add IR LED driver transistor
Parts:
- added Q1: MMBT3904, Librray:SOT-23, B.Cu at (83.8, 83.8)
- added R1: 15, Librray:R_0402_1005Metric, B.Cu at (81.9, 82.5)
- added R2: 2.7k, Librray:R_0402_1005Metric, B.Cu at (86.4, 85.0)
Connections:
- D1 pad 2: Net-(D1-Pad2) -> +3V0
