File: IR-Controller/Hardware/IR-Controller.kicad_pcb (KiCad board)
At the start: 2 copper layers, 7 parts, among them Q1 MMBT3904, U1 PIC18LF2550

Commit message: Refactor library
Split it into smaller files, which contains components related to each
other.

The goal is to make the library reusable across projects.

The resistors and capacitors are still only generic symbols in the
library and it is still up to designer to link to DigiKey. With time
those components will become accessible via library as well.
Parts:
- BT1: footprint Librray:BC-2003 -> Connector_Battery:BC-2003
- C1: footprint Librray:C_0402_1005Metric -> Capacitor_Ceramic:C_0402_1005Metric
- D1: footprint Librray:IN-S126ESGHIR -> LED:IN-S126ESGHIR
- Q1: value MMBT3904 -> MMBT3904LT1G; footprint Librray:SOT-23 -> Package_TO_SOT:SOT-23
- R1, R2: footprint Librray:R_0402_1005Metric -> Resistor:R_0402_1005Metric
- U1: value PIC18LF2550 -> PIC18LF2550-ISO; footprint Librray:SOIC-28_Width7.50mm_Pitch1.27mm -> Package_SO:SOIC-28_Width7.50mm_Pitch1.27mm
