File: IR-Controller/Hardware/IR-Controller.sch (KiCad schematic (older format))
At the start: 7 parts, among them Q1 MMBT3904, U1 PIC18LF2550

Commit message: Refactor library
Split it into smaller files, which contains components related to each
other.

The goal is to make the library reusable across projects.

The resistors and capacitors are still only generic symbols in the
library and it is still up to designer to link to DigiKey. With time
those components will become accessible via library as well.
Parts:
- BT1: footprint Librray:BC-2003 -> Connector_Battery:BC-2003; symbol Library:Battery -> Connector_Battery:BC-2003; Description Battery Retainer Coin, 20.0mm 1 Cell SMD (SMT) Tab -> BATTERY HOLDER COIN 20MM SMD; Detailed Description (none) -> Battery Retainer Coin, 20.0mm 1 Cell SMD (SMT) Tab; Drawing (none) -> https://www.memoryprotectiondevices.com/datasheets/BC-2003-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
- C1: footprint Librray:C_0402_1005Metric -> Capacitor_Ceramic:C_0402_1005Metric; symbol Library:C -> Capacitor_Ceramic:C
- D1: footprint Librray:IN-S126ESGHIR -> LED:IN-S126ESGHIR; symbol Library:LED -> LED:IN-S126ESGHIR; Detailed Description (none) -> Infrared (IR) Emitter 940nm 1.46V 100mA 92mW/sr @ 100mA (Ty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
- Q1: value MMBT3904 -> MMBT3904LT1G; footprint Librray:SOT-23 -> Package_TO_SOT:SOT-23; symbol Library:NPN_BEC -> Transistor_BJT:MMBT3904LT1G; Base Part Number (none) -> MMBT3904; Detailed Description (none) -> Bipolar (BJT) Transistor NPN 40V 200mA 300MHz 300mW Surface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
- R1, R2: footprint Librray:R_0402_1005Metric -> Resistor:R_0402_1005Metric; symbol Library:R -> Resistor:R
- U1: value PIC18LF2550 -> PIC18LF2550-ISO; footprint Librray:SOIC-28_Width7.50mm_Pitch1.27mm -> Package_SO:SOIC-28_Width7.50mm_Pitch1.27mm; symbol Library:PIC18F2550 -> Microcontroller:PIC18LF2550-ISO; Detailed Description (none) -> PIC PIC® 18F Microcontroller IC 8-Bit 48MHz 32KB (16K x 16)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; Digi-Key Part Number PIC18LF2550-I/SO-ND -> PIC18F2550T-I/SOCT-ND; Manufacturer Part Number PIC18LF2550-I/SO -> PIC18F2550T-I/SO
Changed lines of the file:
@@
 $EndDescr
 $Comp
-L Library:PIC18F2550 U1
+L Microcontroller:PIC18LF2550-ISO U1
 U 1 1 6002E7CC
 P 4250 3050
 F 0 "U1" H 5150 4000 50  0000 L BNN
-F 1 "PIC18LF2550" H 5150 3900 50  0000 L BNN
-F 2 "Librray:SOIC-28_Width7.50mm_Pitch1.27mm" H 5700 4000 50  0001 C CNN
-F 3 "${KIPRJMOD}/../../Datasheet/PIC18F2455-2550-4455-4550 Data Sheet.pdf" H 6100 4300 50  0001 C CNN
-F 4 "IC MCU 8BIT 32KB FLASH 28SOIC" H 4650 3350 50  0001 C CNN "Description"
-F 5 "Microchip Technology" H 4650 3350 50  0001 C CNN "Manufacturer"
-F 6 "PIC18LF2550-I/SO" H 4650 3350 50  0001 C CNN "Manufacturer Part Number"
-F 7 "PIC18LF2550-I/SO-ND" H 4650 3350 50  0001 C CNN "Digi-Key Part Number"
+F 1 "PIC18LF2550-ISO" H 5150 3900 50  0000 L BNN
+F 2 "Package_SO:SOIC-28_Width7.50mm_Pitch1.27mm" H 5700 4000 50  0001 C CNN
+F 3 "https://ww1.microchip.com/downloads/en/DeviceDoc/39632e.pdf" H 6100 4300 50  0001 C CNN
+F 4 "IC MCU 8BIT 32KB FLASH 28SOIC" H 4250 3050 50  0001 C CNN "Description"
+F 5 "PIC PIC® 18F Microcontroller IC 8-Bit 48MHz 32KB (16K x 16) FLASH 28-SOIC" H 4250 3050 50  0001 C CNN "Detailed Description"
+F 6 "PIC18F2550T-I/SOCT-ND" H 4250 3050 50  0001 C CNN "Digi-Key Part Number"
+F 7 "Microchip Technology" H 4250 3050 50  0001 C CNN "Manufacturer"
+F 8 "PIC18F2550T-I/SO" H 4250 3050 50  0001 C CNN "Manufacturer Part Number"
 	1    4250 3050
 	1    0    0    -1
@@
 	4250 2050 4250 2150
 $Comp
-L Library:Battery BT1
+L Connector_Battery:BC-2003 BT1
 U 1 1 60036241
 P 1550 1600
 F 0 "BT1" H 1703 1596 50  0000 L CNN
 F 1 "BC-2003" H 1703 1505 50  0000 L CNN
-F 2 "Librray:BC-2003" H 1550 1600 50  0001 C CNN
-F 3 "${KIPRJMOD}/../../Datasheet/BC-2003.pdf" H 1550 1600 50  0001 C CNN
-F 4 "Battery Retainer Coin, 20.0mm 1 Cell SMD (SMT) Tab" H 1550 1600 50  0001 C CNN "Description"
-F 5 "MPD (Memory Protection Devices)" H 1550 1600 50  0001 C CNN "Manufacturer"
-F 6 "BC-2003" H 1550 1600 50  0001 C CNN "Manufacturer Part Number"
-F 7 "BC-2003-ND" H 1550 1600 50  0001 C CNN "Digi-Key Part Number"
+F 2 "Connector_Battery:BC-2003" H 1550 1600 50  0001 C CNN
+F 3 "https://media.digikey.com/pdf/Data%20Sheets/Memory%20Protection%20PDFs/Coin_Cell_Guide.pdf" H 1550 1600 50  0001 C CNN
+F 4 "BATTERY HOLDER COIN 20MM SMD" H 1550 1600 50  0001 C CNN "Description"
+F 5 "Battery Retainer Coin, 20.0mm 1 Cell SMD (SMT) Tab" H 1550 1600 50  0001 C CNN "Detailed Description"
+F 6 "BC-2003-ND" H 1550 1600 50  0001 C CNN "Digi-Key Part Number"
+F 7 "https://www.memoryprotectiondevices.com/datasheets/BC-2003-datasheet.pdf" H 1550 1600 50  0001 C CNN "Drawing"
+F 8 "MPD (Memory Protection Devices)" H 1550 1600 50  0001 C CNN "Manufacturer"
+F 9 "BC-2003" H 1550 1600 50  0001 C CNN "Manufacturer Part Number"
 	1    1550 1600
 	1    0    0    -1
@@
 	1550 1800 1550 1850
 $Comp
-L Library:C C1
+L Capacitor_Ceramic:C C1
 U 1 1 5FE20484
 P 3550 1550
 F 0 "C1" V 3571 1415 50  0000 R CNN
 F 1 "0.1uF" V 3480 1415 50  0000 R CNN
-F 2 "Librray:C_0402_1005Metric" H 3400 1750 50  0001 C CNN
+F 2 "Capacitor_Ceramic:C_0402_1005Metric" H 3400 1750 50  0001 C CNN
 F 3 "" H 3400 1750 50  0001 C CNN
 F 4 "CAP CER 0.1UF 25V X7R 0402" V 3550 1550 50  0001 C CNN "Description"
@@
 	3550 1750 3550 1700
 $Comp
-L Library:NPN_BEC Q1
+L Transistor_BJT:MMBT3904LT1G Q1
 U 1 1 5FE4DCB4
 P 1650 3600
-F 0 "Q1" H 1600 3800 50  0000 R BNN
-F 1 "MMBT3904" H 1600 3700 50  0000 R BNN
-F 2 "Librray:SOT-23" H 1650 3600 50  0001 C CNN
-F 3 "${KIPRJMOD}/../../Datasheet/MMBT3904L SMMBT3904L General Purpose Transistor NPN Silicon.pdf" H 1650 3600 50  0001 C CNN
-F 4 "TRANS NPN 40V 200MA SOT23-3" H 1650 3600 50  0001 C CNN "Description"
-F 5 "ON Semiconductor" H 1650 3600 50  0001 C CNN "Manufacturer"
-F 6 "MMBT3904LT1G" H 1650 3600 50  0001 C CNN "Manufacturer Part Number"
+F 0 "Q1" H 1500 3800 50  0000 L BNN
+F 1 "MMBT3904LT1G" H 1840 3600 50  0001 L BNN
+F 2 "Package_TO_SOT:SOT-23" H 1650 3600 50  0001 C CNN
+F 3 "https://www.onsemi.com/pdf/datasheet/mmbt3904lt1-d.pdf" H 1650 3600 50  0001 C CNN
+F 4 "MMBT3904" H 1200 3700 50  0000 L BNN "Base Part Number"
+F 5 "TRANS NPN 40V 200MA SOT23-3" H 1650 3600 50  0001 C CNN "Description"
+F 6 "Bipolar (BJT) Transistor NPN 40V 200mA 300MHz 300mW Surface Mount SOT-23-3 (TO-236)" H 1650 3600 50  0001 C CNN "Detailed Description"
 F 7 "MMBT3904LT1GOSCT-ND" H 1650 3600 50  0001 C CNN "Digi-Key Part Number"
+F 8 "ON Semiconductor" H 1650 3600 50  0001 C CNN "Manufacturer"
+F 9 "MMBT3904LT1G" H 1650 3600 50  0001 C CNN "Manufacturer Part Number"
 	1    1650 3600
 	-1   0    0    -1
 $EndComp
 $Comp
-L Library:LED D1
+L LED:IN-S126ESGHIR D1
 U 1 1 60035D25
 P 1550 2850
 F 0 "D1" V 1550 2700 50  0000 R TNN
-F 1 "IN-S126ESGHIR" V 1450 2700 50  0000 R TNN
-F 2 "Librray:IN-S126ESGHIR" H 1560 3000 50  0001 C CNN
-F 3 "${KIPRJMOD}/../../Datasheet/IN-S126ESGHIR.pdf" H 1560 3000 50  0001 C CNN
-F 4 "SIDE VIEW / 1210 / 3.0X2.55X1.6" V 1550 2850 50  0001 C CNN "Description"
-F 5 "Inolux" V 1550 2850 50  0001 C CNN "Manufacturer"
-F 6 "IN-S126ESGHIR" V 1550 2850 50  0001 C CNN "Manufacturer Part Number"
-F 7 "1830-IN-S126ESGHIRCT-ND" V 1550 2850 50  0001 C CNN "Digi-Key Part Number"
+F 1 "IN-S126ESGHIR" H 1550 2725 50  0001 C CNN
+F 2 "LED:IN-S126ESGHIR" H 1560 3000 50  0001 C CNN
+F 3 "http://www.inolux-corp.com/datasheet/IR/Emitter/940%20nm%20SMD/IN-S126ESGHIR_V1.1.pdf" H 1560 3000 50  0001 C CNN
+F 4 "SIDE VIEW / 1210 / 3.0X2.55X1.6" H 1550 2850 50  0001 C CNN "Description"
+F 5 "Inolux" H 1550 2850 50  0001 C CNN "Manufacturer"
+F 6 "IN-S126ESGHIR" H 1550 2850 50  0001 C CNN "Manufacturer Part Number"
+F 7 "1830-IN-S126ESGHIRCT-ND" H 1550 2850 50  0001 C CNN "Digi-Key Part Number"
+F 8 "Infrared (IR) Emitter 940nm 1.46V 100mA 92mW/sr @ 100mA (Typ) 30° 1210 (3225 Metric)" H 1550 2850 50  0001 C CNN "Detailed Description"
 	1    1550 2850
 	0    -1   -1   0
@@
 	1550 3800 1550 3850
 $Comp
-L Library:R R?
+L Resistor:R R1
 U 1 1 5FE58D04
 P 1450 3200
-AR Path="/5FE20DA8/5FE58D04" Ref="R?"  Part="1"
-AR Path="/5FE379B8/5FE58D04" Ref="R?"  Part="1"
-AR Path="/5FE58D04" Ref="R1"  Part="1"
 F 0 "R1" H 1200 3150 50  0000 R TNN
 F 1 "15" H 1200 3250 50  0000 R TNN
-F 2 "Librray:R_0402_1005Metric" H 1450 3200 50  0001 C CNN
+F 2 "Resistor:R_0402_1005Metric" H 1450 3200 50  0001 C CNN
 F 3 "" H 1450 3200 50  0001 C CNN
 F 4 "CRGCQ 0402 15R 1%" H 1450 3200 50  0001 C CNN "Description"
@@
 	1550 2650 1550 2700
 $Comp
-L Library:R R?
+L Resistor:R R2
 U 1 1 60036624
 P 2300 3500
-AR Path="/5FE20DA8/60036624" Ref="R?"  Part="1"
-AR Path="/5FE379B8/60036624" Ref="R?"  Part="1"
-AR Path="/60036624" Ref="R2"  Part="1"
 F 0 "R2" V 2050 3550 50  0000 R TNN
 F 1 "2.7k" V 1950 3550 50  0000 R TNN
-F 2 "Librray:R_0402_1005Metric" H 2300 3500 50  0001 C CNN
+F 2 "Resistor:R_0402_1005Metric" H 2300 3500 50  0001 C CNN
 F 3 "" H 2300 3500 50  0001 C CNN
 F 4 "CRGCQ 0402 2K7 1%" H 2300 3500 50  0001 C CNN "Description"
