File: IR-Digipot/hardware/Audio.sch (KiCad schematic (older format))
At the start: 49 parts, among them J3 STX-3500-5NTR, J4 STX-3500-5NTR, Q1 MMBT3904LT1G, Q2 MMBT3906LT1G, Q3 MMBT3904LT1G, Q4 MMBT3906LT1G, U4 OPA2134UA_2K5, U5 OPA2134UA_2K5, U6 AD5262BRUZ50-RL7

Commit message: Add diode between power monitor and MCLR
Should protect the monitor from HV programming.
Will also avoid possible scenario when the monitor will attempt
ti pull MCLR low during programming.
Parts:
- renumbered D3 to D4, D4 to D5
Changed lines of the file:
@@
 Connection ~ 3050 3700
 $Comp
-L Diode:D D3
+L Diode:D D4
 U 1 1 5FFD0310
 P 3150 4650
-F 0 "D3" V 3150 4550 50  0000 R CNN
+F 0 "D4" V 3150 4550 50  0000 R CNN
 F 1 "1N914" V 3050 4550 50  0000 R CNN
 F 2 "Diode:SOD-523" H 3160 4800 50  0001 C CNN
@@
 	3800 5750 3800 5950
 $Comp
-L Diode:D D4
+L Diode:D D5
 U 1 1 5FFEA13D
 P 3150 6750
-F 0 "D4" V 3150 6650 50  0000 R CNN
+F 0 "D5" V 3150 6650 50  0000 R CNN
 F 1 "1N914" V 3050 6650 50  0000 R CNN
 F 2 "Diode:SOD-523" H 3160 6900 50  0001 C CNN
