File: IR-Digipot/hardware/CPU.sch (KiCad schematic (older format))
At the start: 18 parts, among them J1 Conn_1x06_Generic, J2 Conn_1x03_Generic, U1 TCM809LVNB713, U2 PIC18F2550T-ISO, U3 TSOP75438TR, X1 ABM8W-20.0000MHZ-4-K1Z-T3

Commit message: Add diode between power monitor and MCLR
Should protect the monitor from HV programming.
Will also avoid possible scenario when the monitor will attempt
ti pull MCLR low during programming.
Parts:
- added D1: SS14HE, Diode:SOD-323HE, symbol Diode:SS14HE
- renumbered D1 to D2, D2 to D3
Connections:
- net MCLR: now also D1.1; no longer R1.1, U1.2 (~RESET~)
- new net: D1.2, R1.1, U1.2 (~RESET~)
Other:
- moved on the sheet: R1, U1
Changed lines of the file:
@@
 $EndComp
 $Comp
-L power:GNDD #PWR03
+L power:GNDD #PWR05
 U 1 1 5FE2F103
 P 2100 4100
-F 0 "#PWR03" H 2100 3850 50  0001 C CNN
+F 0 "#PWR05" H 2100 3850 50  0001 C CNN
 F 1 "GNDD" H 2104 3945 50  0000 C CNN
 F 2 "" H 2100 4100 50  0001 C CNN
@@
 	6000 4850 6000 5100
 $Comp
-L LED:HSMG-C170 D2
+L LED:HSMG-C170 D3
 U 1 1 6018F3C2
 P 6350 5600
-F 0 "D2" V 6450 5650 50  0000 L CNN
+F 0 "D3" V 6450 5650 50  0000 L CNN
 F 1 "HSMG-C170" H 6350 5475 50  0001 C CNN
 F 2 "LED:HSMx-C170" H 6360 5750 50  0001 C CNN
@@
 	6350 5400 6350 5450
 $Comp
-L LED:HSMG-C170 D1
+L LED:HSMG-C170 D2
 U 1 1 60180CAB
 P 6000 5600
-F 0 "D1" V 6100 5650 50  0000 L CNN
+F 0 "D2" V 6100 5650 50  0000 L CNN
 F 1 "HSMG-C170" H 6000 5475 50  0001 C CNN
 F 2 "LED:HSMx-C170" H 6010 5750 50  0001 C CNN
@@
 $EndComp
 Wire Wire Line
-	2750 2150 2750 2250
-Wire Wire Line
-	2750 1800 3050 1800
-Connection ~ 2750 1800
-Wire Wire Line
-	2750 1850 2750 1800
-Wire Wire Line
-	2650 1800 2750 1800
-Wire Wire Line
-	2200 2150 2200 2250
+	2400 2150 2400 2250
+Wire Wire Line
+	2400 1800 2700 1800
+Connection ~ 2400 1800
+Wire Wire Line
+	2400 1850 2400 1800
+Wire Wire Line
+	2300 1800 2400 1800
+Wire Wire Line
+	1850 2150 1850 2250
 $Comp
 L power:GNDD #PWR06
 U 1 1 5FE43D04
-P 2750 2250
-F 0 "#PWR06" H 2750 2000 50  0001 C CNN
-F 1 "GNDD" H 2754 2095 50  0000 C CNN
-F 2 "" H 2750 2250 50  0001 C CNN
-F 3 "" H 2750 2250 50  0001 C CNN
-	1    2750 2250
+P 2400 2250
+F 0 "#PWR06" H 2400 2000 50  0001 C CNN
+F 1 "GNDD" H 2404 2095 50  0000 C CNN
+F 2 "" H 2400 2250 50  0001 C CNN
+F 3 "" H 2400 2250 50  0001 C CNN
+	1    2400 2250
 	1    0    0    -1
 $EndComp
@@
 L Resistor:R R1
 U 1 1 5FE4251D
-P 2850 2000
-F 0 "R1" H 2820 2046 50  0000 L CNN
-F 1 "100K" H 2820 1955 50  0000 L CNN
-F 2 "Resistor:R_0402_1005Metric" H 2850 2000 50  0001 C CNN
-F 3 "" H 2850 2000 50  0001 C CNN
-F 4 "CRGCQ 0402 100K 1%" H 2850 2000 50  0001 C CNN "Description"
-F 5 "TE Connectivity Passive Product" H 2850 2000 50  0001 C CNN "Manufacturer"
-F 6 "CRGCQ0402F100K" H 2850 2000 50  0001 C CNN "Manufacturer Part Number"
-F 7 "A129651CT-ND" H 2850 2000 50  0001 C CNN "Digi-Key Part Number"
-	1    2850 2000
-	1    0    0    -1
-$EndComp
-Wire Wire Line
-	2200 1400 2200 1450
-$Comp
-L power:GNDD #PWR05
+P 2500 2000
+F 0 "R1" H 2470 2046 50  0000 L CNN
+F 1 "100K" H 2470 1955 50  0000 L CNN
+F 2 "Resistor:R_0402_1005Metric" H 2500 2000 50  0001 C CNN
+F 3 "" H 2500 2000 50  0001 C CNN
+F 4 "CRGCQ 0402 100K 1%" H 2500 2000 50  0001 C CNN "Description"
+F 5 "TE Connectivity Passive Product" H 2500 2000 50  0001 C CNN "Manufacturer"
+F 6 "CRGCQ0402F100K" H 2500 2000 50  0001 C CNN "Manufacturer Part Number"
+F 7 "A129651CT-ND" H 2500 2000 50  0001 C CNN "Digi-Key Part Number"
+	1    2500 2000
+	1    0    0    -1
+$EndComp
+Wire Wire Line
+	1850 1400 1850 1450
+$Comp
+L power:GNDD #PWR04
 U 1 1 5FE2B9AA
-P 2200 2250
-F 0 "#PWR05" H 2200 2000 50  0001 C CNN
-F 1 "GNDD" H 2204 2095 50  0000 C CNN
-F 2 "" H 2200 2250 50  0001 C CNN
-F 3 "" H 2200 2250 50  0001 C CNN
-	1    2200 2250
-	1    0    0    -1
-$EndComp
-$Comp
-L power:+5VD #PWR04
+P 1850 2250
+F 0 "#PWR04" H 1850 2000 50  0001 C CNN
+F 1 "GNDD" H 1854 2095 50  0000 C CNN
+F 2 "" H 1850 2250 50  0001 C CNN
+F 3 "" H 1850 2250 50  0001 C CNN
+	1    1850 2250
+	1    0    0    -1
+$EndComp
+$Comp
+L power:+5VD #PWR03
 U 1 1 5FE2B259
-P 2200 1400
-F 0 "#PWR04" H 2200 1250 50  0001 C CNN
-F 1 "+5VD" H 2215 1573 50  0000 C CNN
-F 2 "" H 2200 1400 50  0001 C CNN
-F 3 "" H 2200 1400 50  0001 C CNN
-	1    2200 1400
+P 1850 1400
+F 0 "#PWR03" H 1850 1250 50  0001 C CNN
+F 1 "+5VD" H 1865 1573 50  0000 C CNN
+F 2 "" H 1850 1400 50  0001 C CNN
+F 3 "" H 1850 1400 50  0001 C CNN
+	1    1850 1400
 	1    0    0    -1
 $EndComp
@@
 L Power_Supervisor:TCM809LVNB713 U1
 U 1 1 5FE25880
-P 2200 1750
-F 0 "U1" H 2072 1746 50  0000 R CNN
-F 1 "TCM809LVNB713" H 2072 1655 50  0000 R CNN
-F 2 "Package_TO_SOT:SOT-23" H 2650 1950 50  0001 C CNN
-F 3 "https://ww1.microchip.com/downloads/en/DeviceDoc/21661E.pdf" H 2650 1950 50  0001 C CNN
-F 4 "IC SUPERVISOR 1 CHANNEL SOT23-3" H 2200 1750 50  0001 C CNN "Description"
-F 5 "Supervisor Push-Pull, Totem Pole 1 Channel SOT-23-3" H 2200 1750 50  0001 C CNN "Detailed Description"
-F 6 "TCM809LVNB713CT-ND" H 2200 1750 50  0001 C CNN "Digi-Key Part Number"
-F 7 "Microchip Technology" H 2200 1750 50  0001 C CNN "Manufacturer"
-F 8 "TCM809LVNB713" H 2200 1750 50  0001 C CNN "Manufacturer Part Number"
-	1    2200 1750
-	1    0    0    -1
-$EndComp
+P 1850 1750
+F 0 "U1" H 1722 1746 50  0000 R CNN
+F 1 "TCM809LVNB713" H 1722 1655 50  0000 R CNN
+F 2 "Package_TO_SOT:SOT-23" H 2300 1950 50  0001 C CNN
+F 3 "https://ww1.microchip.com/downloads/en/DeviceDoc/21661E.pdf" H 2300 1950 50  0001 C CNN
+F 4 "IC SUPERVISOR 1 CHANNEL SOT23-3" H 1850 1750 50  0001 C CNN "Description"
+F 5 "Supervisor Push-Pull, Totem Pole 1 Channel SOT-23-3" H 1850 1750 50  0001 C CNN "Detailed Description"
+F 6 "TCM809LVNB713CT-ND" H 1850 1750 50  0001 C CNN "Digi-Key Part Number"
+F 7 "Microchip Technology" H 1850 1750 50  0001 C CNN "Manufacturer"
+F 8 "TCM809LVNB713" H 1850 1750 50  0001 C CNN "Manufacturer Part Number"
+	1    1850 1750
+	1    0    0    -1
+$EndComp
+$Comp
+L Diode:SS14HE D1
+U 1 1 60460A64
+P 2850 1800
+F 0 "D1" H 2850 1585 50  0000 C CNN
+F 1 "SS14HE" H 2850 1676 50  0000 C CNN
+F 2 "Diode:SOD-323HE" H 2860 1950 50  0001 C CNN
+F 3 "https://www.onsemi.com/pdf/datasheet/ss13he-d.pdf" H 2860 1950 50  0001 C CNN
+F 4 "DIODE SCHOTTKY 40V 1A SOD323HE" H 2850 1800 50  0001 C CNN "Description"
+F 5 "Diode Schottky 40V 1A Surface Mount SOD-323HE" H 2850 1800 50  0001 C CNN "Detailed Description"
+F 6 "ON Semiconductor" H 2850 1800 50  0001 C CNN "Manufacturer"
+F 7 "SS14HE" H 2850 1800 50  0001 C CNN "Manufacturer Part Number"
+F 8 "SS14HECT-ND" H 2850 1800 50  0001 C CNN "Digi-Key Part Number"
+F 9 "SS14" H 2850 1800 50  0001 C CNN "Base Part Number"
+	1    2850 1800
+	-1   0    0    1
+$EndComp
+Wire Wire Line
+	3000 1800 3050 1800
 $EndSCHEMATC
