File: IR-Digipot/hardware/Power Delivery.sch (KiCad schematic (older format))
At the start: 26 parts, among them J5 1054500101, Q5 STL6P3LLH6, Q6 STL6P3LLH6, U7 STUSB4500QTR

Commit message: Add diode between power monitor and MCLR
Should protect the monitor from HV programming.
Will also avoid possible scenario when the monitor will attempt
ti pull MCLR low during programming.
Parts:
- renumbered D5 to D6, D6 to D7, D7 to D8, D8 to D9
Changed lines of the file:
@@
 	2400 4150 2400 4200
 $Comp
-L Diode:D_ZENNER D5
+L Diode:D_ZENNER D6
 U 1 1 5FF29B69
 P 2850 4000
-F 0 "D5" V 2804 4078 50  0000 L CNN
+F 0 "D6" V 2804 4078 50  0000 L CNN
 F 1 "ESDA25P35" V 2895 4078 50  0000 L CNN
 F 2 "Package_DFN_QFN:UDFN-2" H 2860 4150 50  0001 C CNN
@@
 $EndComp
 $Comp
-L Diode:D_ZENNER_DUAL_CATHODE D6
+L Diode:D_ZENNER_DUAL_CATHODE D7
 U 1 1 5FF329A1
 P 3550 5050
-F 0 "D6" V 3504 5128 50  0000 L CNN
+F 0 "D7" V 3504 5128 50  0000 L CNN
 F 1 "ESDA25W" V 3595 5128 50  0000 L CNN
 F 2 "Package_TO_SOT:SOT-323" H 3560 5200 50  0001 C CNN
@@
 $EndComp
 $Comp
-L Diode:D_SCHOTTKY D7
+L Diode:D_SCHOTTKY D8
 U 1 1 5FE776B2
 P 5400 1850
-F 0 "D7" V 5450 2150 50  0000 R CNN
+F 0 "D8" V 5450 2150 50  0000 R CNN
 F 1 "BAT54" V 5350 2150 50  0000 R CNN
 F 2 "Diode:SOD-523" H 5410 2000 50  0001 C CNN
@@
 	7900 3450 7900 4000
 $Comp
-L Diode:D_ZENNER D8
+L Diode:D_ZENNER D9
 U 1 1 5FEF03A0
 P 9400 2700
-F 0 "D8" V 9354 2778 50  0000 L CNN
+F 0 "D9" V 9354 2778 50  0000 L CNN
 F 1 "ESDA25P35" V 9445 2778 50  0000 L CNN
 F 2 "Package_DFN_QFN:UDFN-2" H 9410 2850 50  0001 C CNN
