File: IR-Digipot/hardware/Power.sch (KiCad schematic (older format))
At the start: 40 parts, among them Q7 STL6P3LLH6, U8 L7985TR, U9 LM27761DSGR

Commit message: Use proper Schottky diode
There was a discontinuity between component value and DigiKey part
number. Use SS14 diode, which is more generic.
Parts:
- D9: value STPS3L60U -> SS14HE; symbol Diode:D_SCHOTTKY -> Diode:SS14HE; Base Part Number (none) -> SS14; Detailed Description (none) -> Diode Schottky 40V 1A Surface Mount SOD-323HE
Changed lines of the file:
@@
 Connection ~ 4100 2350
 $Comp
-L Diode:D_SCHOTTKY D9
+L Diode:SS14HE D9
 U 1 1 5FEA0696
 P 3850 1650
-F 0 "D9" V 3804 1728 50  0000 L CNN
-F 1 "STPS3L60U" V 3895 1728 50  0000 L CNN
+F 0 "D9" V 3800 1750 50  0000 L CNN
+F 1 "SS14HE" V 3900 1750 50  0000 L BNN
 F 2 "Diode:SOD-323HE" H 3860 1800 50  0001 C CNN
-F 3 "" H 3860 1800 50  0001 C CNN
-F 4 "DIODE SCHOTTKY 40V 1A SOD323HE" V 3850 1650 50  0001 C CNN "Description"
-F 5 "ON Semiconductor" V 3850 1650 50  0001 C CNN "Manufacturer"
-F 6 "SS14HE" V 3850 1650 50  0001 C CNN "Manufacturer Part Number"
-F 7 "SS14HECT-ND" V 3850 1650 50  0001 C CNN "Digi-Key Part Number"
+F 3 "https://www.onsemi.com/pdf/datasheet/ss13he-d.pdf" H 3860 1800 50  0001 C CNN
+F 4 "DIODE SCHOTTKY 40V 1A SOD323HE" H 3850 1650 50  0001 C CNN "Description"
+F 5 "ON Semiconductor" H 3850 1650 50  0001 C CNN "Manufacturer"
+F 6 "SS14HE" H 3850 1650 50  0001 C CNN "Manufacturer Part Number"
+F 7 "SS14HECT-ND" H 3850 1650 50  0001 C CNN "Digi-Key Part Number"
+F 8 "SS14" H 3850 1650 50  0001 C CNN "Base Part Number"
+F 9 "Diode Schottky 40V 1A Surface Mount SOD-323HE" H 3850 1650 50  0001 C CNN "Detailed Description"
 	1    3850 1650
 	0    1    1    0

Commit message: Add diode between power monitor and MCLR
Should protect the monitor from HV programming.
Will also avoid possible scenario when the monitor will attempt
ti pull MCLR low during programming.
Parts:
- renumbered D9 to D10, D10 to D11
Changed lines of the file:
@@
 Connection ~ 4100 2350
 $Comp
-L Diode:SS14HE D9
+L Diode:SS14HE D10
 U 1 1 5FEA0696
 P 3850 1650
-F 0 "D9" V 3800 1750 50  0000 L CNN
+F 0 "D10" V 3800 1750 50  0000 L CNN
 F 1 "SS14HE" V 3900 1750 50  0000 L BNN
 F 2 "Diode:SOD-323HE" H 3860 1800 50  0001 C CNN
@@
 Connection ~ 4900 1450
 $Comp
-L Diode:D_ZENNER D10
+L Diode:D_ZENNER D11
 U 1 1 5FE73A35
 P 5900 1750
-F 0 "D10" V 5854 1828 50  0000 L CNN
+F 0 "D11" V 5854 1828 50  0000 L CNN
 F 1 "ESDA7P120" V 5945 1828 50  0000 L CNN
 F 2 "Diode:D_0603_1610Metric" H 5910 1900 50  0001 C CNN
