File: IR-Digipot/hardware/IR Digipot.kicad_pcb (KiCad board)
At the start: 2 copper layers, 54.9 x 58.4 mm, 133 parts, among them J1 Conn_1x06_Generic, J2 Conn_1x03_Generic, J3 STX-3500-5NTR, J4 STX-3500-5NTR, J5 1054500101, Q1 MMBT3904LT1G, Q2 MMBT3906LT1G, Q3 MMBT3904LT1G, Q4 MMBT3906LT1G, Q5 STL6P3LLH6, Q6 STL6P3LLH6, Q7 STL6P3LLH6, U1 TCM809LVNB713, U2 PIC18F2550T-ISO, U3 TSOP75438TR, U4 OPA2134UA_2K5, U5 OPA2134UA_2K5, U6 AD5262BRUZ50-RL7, U7 STUSB4500QTR, U8 L7985TR, U9 LM27761DSGR, X1 ABM8W-20.0000MHZ-4-K1Z-T3

Commit message: Use proper Schottky diode
There was a discontinuity between component value and DigiKey part
number. Use SS14 diode, which is more generic.
Parts:
- D9: value STPS3L60U -> SS14HE
Changed lines of the file:
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@@
       (effects (font (size 0.6 0.6) (thickness 0.15)))
     )
-    (fp_text value STPS3L60U (at 0 1.524 90) (layer F.Fab)
+    (fp_text value SS14HE (at 0 1.524 90) (layer F.Fab)
       (effects (font (size 1 1) (thickness 0.15)))
     )

Commit message: Add diode between power monitor and MCLR
Should protect the monitor from HV programming.
Will also avoid possible scenario when the monitor will attempt
ti pull MCLR low during programming.
Parts:
- added D1: SS14HE, Diode:SOD-323HE, F.Cu at (121.7, 78.9)
- moved R1 5.54 mm to (118.5, 82.0), turned to 180 degrees
- moved U1 1.43 mm to (119.1, 79.7), turned to 90 degrees
- renumbered D9 to D10, D10 to D11, D1 to D2, D2 to D3, D3 to D4, D4 to D5, D5 to D6, D6 to D7, D7 to D8, D8 to D9
Connections:
- R1 pad 1: /CPU/MCLR -> Net-(D1-Pad2)
- U1 pad 2: /CPU/MCLR -> Net-(D1-Pad2)
Routing:
- net Net-(D1-Pad2): track 0.00 -> 3.53 mm

Commit message: Digipot: Move labels to the copper layer
Should make it look better with the manufacturing process.
Routing:
- net DIGIPOT_SHDN: track 37.4 -> 38.2 mm
- net SPI_CLK: track 22.3 -> 23.1 mm
- net SPI_MOSI: track 22.6 -> 23.3 mm
- net SPI_CS_DIGIPOT: track 26.7 -> 27.3 mm
Other:
- board text added: "May, 2021"
- board text removed: "Jan, 2021"
