File: IR-Controller/hardware/IR-Controller.sch (KiCad schematic (older format))
At the start: 7 parts, among them Q1 MMBT3904LT1G, U1 PIC18LF2550-ISO

Commit message: Initial version of controller suitable for debugging
Parts:
- added J1: Conn_1x06_Generic, Connector_Generic:Conn_1x06_Socket_Pitch2.54mm_sideways, symbol Connector_Generic:Conn_1x06_Generic
- added R3: CRGCQ0402F10K, Resistor:R_0402_1005Metric, symbol Resistor:CRGCQ0402F10K
- added SW1, SW2: MCSLPT4644B1TR, Switches:MCSLPT4644B1TR, symbol Switches:MCSLPT4644B1TR
Connections:
- net GND: now also J1.4, R3.2
- net MCLR: now reaches U1.1 (~MCLR~/VPP/RE3)
- net MCLR: now also J1.6
- net SW_COL_0: now reaches U1.21 (RB0/AN12/INT0/FLT0/SDI/SDA)
- net SW_COL_0: now also R3.1, SW1.1, SW2.1
- net SW_ROW_0: now reaches U1.25 (RB4/AN11/KBI0)
- net SW_ROW_0: now also SW2.2
- net SW_ROW_1: now reaches U1.26 (RB5/KBI1/PGM)
- net SW_ROW_1: now also SW1.2
- net PGC: now reaches U1.27 (RB6/KBI2/PGC)
- net PGC: now also J1.2
- net PGD: now reaches U1.28 (RB7/KBI3/PGD)
- net PGD: now also J1.3
- net +3V0 renamed +3V
- net +3V: now also J1.5

Commit message: Controller: Pull RC4 and RC5 to ground
Those are digital inputs when USB is not used. Pull to ground to avoid
excess power drain.
Connections:
- net GND: now also U1.15 (RC4/D-/VM), U1.16 (RC5/D+/VP)
Other:
- moved on the sheet: R3
Changed lines of the file:
@@
 L Resistor:CRGCQ0402F10K R3
 U 1 1 6069684D
-P 6000 4050
-F 0 "R3" H 5970 4096 50  0000 L CNN
-F 1 "CRGCQ0402F10K" H 5950 4050 50  0001 L BNN
-F 2 "Resistor:R_0402_1005Metric" H 6000 4050 50  0001 C CNN
-F 3 "https://www.te.com/commerce/DocumentDelivery/DDEController?Action=srchrtrv&DocNm=1773204-3&DocType=DS&DocLang=English" H 6000 4050 50  0001 C CNN
-F 4 "CRGCQ 0402 10K 1%" H 6000 4050 50  0001 C CNN "Description"
-F 5 "10 kOhms ±1% 0.063W, 1/16W Chip Resistor 0402 (1005 Metric) Automotive AEC-Q200, Moisture Resistant Thick Film" H 6000 4050 50  0001 C CNN "Detailed Description"
-F 6 "TE Connectivity Passive Product" H 6000 4050 50  0001 C CNN "Manufacturer"
-F 7 "CRGCQ0402F10K" H 6000 4050 50  0001 C CNN "Manufacturer Part Number"
-F 8 "A129639CT-ND" H 6000 4050 50  0001 C CNN "Digi-Key Part Number"
-F 9 "10k" H 5970 4005 50  0000 L CNN "Resistance"
-F 10 "CRGCQ" H 6000 4050 50  0001 C CNN "Series"
-F 11 "Cut Tape (CT)" H 6000 4050 50  0001 C CNN "Packaging"
-F 12 "±1%" H 6000 4050 50  0001 C CNN "Tolerance"
-F 13 "0.063W, 1/16W" H 6000 4050 50  0001 C CNN "Power (Watts)"
-F 14 "Thick Film" H 6000 4050 50  0001 C CNN "Composition"
-F 15 "Automotive AEC-Q200, Moisture Resistant" H 6000 4050 50  0001 C CNN "Features"
-F 16 "±100ppm/°C" H 6000 4050 50  0001 C CNN "Temperature Coefficient"
-F 17 "-55°C ~ 155°C" H 6000 4050 50  0001 C CNN "Operating Temperature"
-F 18 "0402 (1005 Metric)" H 6000 4050 50  0001 C CNN "Package / Case"
-F 19 "AEC-Q200" H 6000 4050 50  0001 C CNN "Ratings"
-F 20 "0402" H 6000 4050 50  0001 C CNN "Supplier Device Package"
-F 21 "0.039\" L x 0.020\" W (1.00mm x 0.50mm)" H 6000 4050 50  0001 C CNN "Size / Dimension"
-F 22 "0.016\" (0.40mm)" H 6000 4050 50  0001 C CNN "Height - Seated (Max)"
-F 23 "2" H 6000 4050 50  0001 C CNN "Number of Terminations"
-F 24 "CRGCQ0402" H 6000 4050 50  0001 C CNN "Base Part Number"
-	1    6000 4050
+P 6350 4050
+F 0 "R3" H 6320 4096 50  0000 L CNN
+F 1 "CRGCQ0402F10K" H 6300 4050 50  0001 L BNN
+F 2 "Resistor:R_0402_1005Metric" H 6350 4050 50  0001 C CNN
+F 3 "https://www.te.com/commerce/DocumentDelivery/DDEController?Action=srchrtrv&DocNm=1773204-3&DocType=DS&DocLang=English" H 6350 4050 50  0001 C CNN
+F 4 "CRGCQ 0402 10K 1%" H 6350 4050 50  0001 C CNN "Description"
+F 5 "10 kOhms ±1% 0.063W, 1/16W Chip Resistor 0402 (1005 Metric) Automotive AEC-Q200, Moisture Resistant Thick Film" H 6350 4050 50  0001 C CNN "Detailed Description"
+F 6 "TE Connectivity Passive Product" H 6350 4050 50  0001 C CNN "Manufacturer"
+F 7 "CRGCQ0402F10K" H 6350 4050 50  0001 C CNN "Manufacturer Part Number"
+F 8 "A129639CT-ND" H 6350 4050 50  0001 C CNN "Digi-Key Part Number"
+F 9 "10k" H 6320 4005 50  0000 L CNN "Resistance"
+F 10 "CRGCQ" H 6350 4050 50  0001 C CNN "Series"
+F 11 "Cut Tape (CT)" H 6350 4050 50  0001 C CNN "Packaging"
+F 12 "±1%" H 6350 4050 50  0001 C CNN "Tolerance"
+F 13 "0.063W, 1/16W" H 6350 4050 50  0001 C CNN "Power (Watts)"
+F 14 "Thick Film" H 6350 4050 50  0001 C CNN "Composition"
+F 15 "Automotive AEC-Q200, Moisture Resistant" H 6350 4050 50  0001 C CNN "Features"
+F 16 "±100ppm/°C" H 6350 4050 50  0001 C CNN "Temperature Coefficient"
+F 17 "-55°C ~ 155°C" H 6350 4050 50  0001 C CNN "Operating Temperature"
+F 18 "0402 (1005 Metric)" H 6350 4050 50  0001 C CNN "Package / Case"
+F 19 "AEC-Q200" H 6350 4050 50  0001 C CNN "Ratings"
+F 20 "0402" H 6350 4050 50  0001 C CNN "Supplier Device Package"
+F 21 "0.039\" L x 0.020\" W (1.00mm x 0.50mm)" H 6350 4050 50  0001 C CNN "Size / Dimension"
+F 22 "0.016\" (0.40mm)" H 6350 4050 50  0001 C CNN "Height - Seated (Max)"
+F 23 "2" H 6350 4050 50  0001 C CNN "Number of Terminations"
+F 24 "CRGCQ0402" H 6350 4050 50  0001 C CNN "Base Part Number"
+	1    6350 4050
 	1    0    0    -1
 $EndComp
@@
 L Power:GND #PWR09
 U 1 1 6069D06B
-P 5900 4250
-F 0 "#PWR09" H 5900 4050 50  0001 C CNN
-F 1 "GND" H 5905 4112 50  0000 C CNN
-F 2 "" H 5900 4250 50  0001 C CNN
-F 3 "" H 5900 4250 50  0001 C CNN
-	1    5900 4250
+P 6250 4250
+F 0 "#PWR09" H 6250 4050 50  0001 C CNN
+F 1 "GND" H 6255 4112 50  0000 C CNN
+F 2 "" H 6250 4250 50  0001 C CNN
+F 3 "" H 6250 4250 50  0001 C CNN
+	1    6250 4250
 	1    0    0    -1
 $EndComp
 Wire Wire Line
-	5900 4200 5900 4250
+	6250 4200 6250 4250
 $Comp
 L Power:+3V #PWR03
@@
 PGC
 Wire Wire Line
-	5650 3100 5900 3100
-Wire Wire Line
 	5650 2600 6750 2600
 Wire Wire Line
 	5650 2700 6750 2700
 Wire Wire Line
-	5900 3100 5900 3900
-Connection ~ 5900 3100
+	6250 3100 6250 3900
+Connection ~ 6250 3100
 Wire Wire Line
-	5900 3100 6750 3100
+	6250 3100 6750 3100
+Wire Wire Line
+	5650 3100 6250 3100
+Wire Wire Line
+	5650 3700 5700 3700
+$Comp
+L Power:GND #PWR?
+U 1 1 6069341C
+P 5700 4250
+F 0 "#PWR?" H 5700 4050 50  0001 C CNN
+F 1 "GND" H 5705 4112 50  0000 C CNN
+F 2 "" H 5700 4250 50  0001 C CNN
+F 3 "" H 5700 4250 50  0001 C CNN
+	1    5700 4250
+	1    0    0    -1
+$EndComp
+Wire Wire Line
+	5650 3600 5900 3600
+$Comp
+L Power:GND #PWR?
+U 1 1 6069472C
+P 5900 4250
+F 0 "#PWR?" H 5900 4050 50  0001 C CNN
+F 1 "GND" H 5905 4112 50  0000 C CNN
+F 2 "" H 5900 4250 50  0001 C CNN
+F 3 "" H 5900 4250 50  0001 C CNN
+	1    5900 4250
+	1    0    0    -1
+$EndComp
+Wire Wire Line
+	5700 3700 5700 4250
+Wire Wire Line
+	5900 3600 5900 4250
 $EndSCHEMATC

Commit message: Controller: Pull MCLR to ground via 10k resistor
When MCLR is used the pin acts as an input. Pull to ground to avoid its
floating state. Use 10k resistor so that the ICSP can still work.

Also update the board.
Parts:
- added R3: CRGCQ0402F10K, Resistor:R_0402_1005Metric, symbol Resistor:CRGCQ0402F10K
- renumbered R3 to R4
Connections:
- net GND: now also R3.2
- net MCLR: now also R3.1
Changed lines of the file:
@@
 $EndComp
 $Comp
-L Power:GND #PWR07
+L Power:GND #PWR08
 U 1 1 60685DB1
 P 4200 4050
-F 0 "#PWR07" H 4200 3850 50  0001 C CNN
+F 0 "#PWR08" H 4200 3850 50  0001 C CNN
 F 1 "GND" H 4205 3912 50  0000 C CNN
 F 2 "" H 4200 4050 50  0001 C CNN
@@
 $EndComp
 $Comp
-L Power:GND #PWR06
+L Power:GND #PWR07
 U 1 1 60686FF1
 P 3550 1750
-F 0 "#PWR06" H 3550 1550 50  0001 C CNN
+F 0 "#PWR07" H 3550 1550 50  0001 C CNN
 F 1 "GND" H 3555 1612 50  0000 C CNN
 F 2 "" H 3550 1750 50  0001 C CNN
@@
 $EndComp
 $Comp
-L Power:+3V #PWR05
+L Power:+3V #PWR06
 U 1 1 60685E70
 P 3550 1350
-F 0 "#PWR05" H 3550 1200 50  0001 C CNN
+F 0 "#PWR06" H 3550 1200 50  0001 C CNN
 F 1 "+3V" H 3565 1523 50  0000 C CNN
 F 2 "" H 3550 1350 50  0001 C CNN
@@
 $EndComp
 $Comp
-L Power:+3V #PWR08
+L Power:+3V #PWR09
 U 1 1 60686867
 P 4250 2050
-F 0 "#PWR08" H 4250 1900 50  0001 C CNN
+F 0 "#PWR09" H 4250 1900 50  0001 C CNN
 F 1 "+3V" H 4265 2223 50  0000 C CNN
 F 2 "" H 4250 2050 50  0001 C CNN
@@
 	7500 2600 7500 2750
 $Comp
-L Resistor:CRGCQ0402F10K R3
+L Resistor:CRGCQ0402F10K R4
 U 1 1 6069684D
 P 6350 4050
-F 0 "R3" H 6320 4096 50  0000 L CNN
+F 0 "R4" H 6320 4096 50  0000 L CNN
 F 1 "CRGCQ0402F10K" H 6300 4050 50  0001 L BNN
 F 2 "Resistor:R_0402_1005Metric" H 6350 4050 50  0001 C CNN
@@
 $EndComp
 $Comp
-L Power:GND #PWR09
+L Power:GND #PWR012
 U 1 1 6069D06B
 P 6250 4250
-F 0 "#PWR09" H 6250 4050 50  0001 C CNN
+F 0 "#PWR012" H 6250 4050 50  0001 C CNN
 F 1 "GND" H 6255 4112 50  0000 C CNN
 F 2 "" H 6250 4250 50  0001 C CNN
@@
 	7700 4200 7700 4600
 $Comp
-L Power:GND #PWR0101
+L Power:GND #PWR014
 U 1 1 6068FA1F
 P 7700 4600
-F 0 "#PWR0101" H 7700 4400 50  0001 C CNN
+F 0 "#PWR014" H 7700 4400 50  0001 C CNN
 F 1 "GND" H 7705 4462 50  0000 C CNN
 F 2 "" H 7700 4600 50  0001 C CNN
@@
 $EndComp
 $Comp
-L Power:+3V #PWR0102
+L Power:+3V #PWR013
 U 1 1 60690747
 P 7650 3650
-F 0 "#PWR0102" H 7650 3500 50  0001 C CNN
+F 0 "#PWR013" H 7650 3500 50  0001 C CNN
 F 1 "+3V" H 7665 3823 50  0000 C CNN
 F 2 "" H 7650 3650 50  0001 C CNN
@@
 $EndComp
 Wire Wire Line
-	2850 2400 2200 2400
+	2850 2400 2450 2400
 Text Label 2200 2400 0    50   ~ 0
 MCLR
@@
 	5650 3700 5700 3700
 $Comp
-L Power:GND #PWR?
+L Power:GND #PWR010
 U 1 1 6069341C
 P 5700 4250
-F 0 "#PWR?" H 5700 4050 50  0001 C CNN
+F 0 "#PWR010" H 5700 4050 50  0001 C CNN
 F 1 "GND" H 5705 4112 50  0000 C CNN
 F 2 "" H 5700 4250 50  0001 C CNN
@@
 	5650 3600 5900 3600
 $Comp
-L Power:GND #PWR?
+L Power:GND #PWR011
 U 1 1 6069472C
 P 5900 4250
-F 0 "#PWR?" H 5900 4050 50  0001 C CNN
+F 0 "#PWR011" H 5900 4050 50  0001 C CNN
 F 1 "GND" H 5905 4112 50  0000 C CNN
 F 2 "" H 5900 4250 50  0001 C CNN
@@
 Wire Wire Line
 	5900 3600 5900 4250
+$Comp
+L Resistor:CRGCQ0402F10K R3
+U 1 1 606960CD
+P 2550 2600
+F 0 "R3" H 2520 2646 50  0000 L CNN
+F 1 "CRGCQ0402F10K" H 2500 2600 50  0001 L BNN
+F 2 "Resistor:R_0402_1005Metric" H 2550 2600 50  0001 C CNN
+F 3 "https://www.te.com/commerce/DocumentDelivery/DDEController?Action=srchrtrv&DocNm=1773204-3&DocType=DS&DocLang=English" H 2550 2600 50  0001 C CNN
+F 4 "CRGCQ 0402 10K 1%" H 2550 2600 50  0001 C CNN "Description"
+F 5 "10 kOhms ±1% 0.063W, 1/16W Chip Resistor 0402 (1005 Metric) Automotive AEC-Q200, Moisture Resistant Thick Film" H 2550 2600 50  0001 C CNN "Detailed Description"
+F 6 "TE Connectivity Passive Product" H 2550 2600 50  0001 C CNN "Manufacturer"
+F 7 "CRGCQ0402F10K" H 2550 2600 50  0001 C CNN "Manufacturer Part Number"
+F 8 "A129639CT-ND" H 2550 2600 50  0001 C CNN "Digi-Key Part Number"
+F 9 "10k" H 2520 2555 50  0000 L CNN "Resistance"
+F 10 "CRGCQ" H 2550 2600 50  0001 C CNN "Series"
+F 11 "Cut Tape (CT)" H 2550 2600 50  0001 C CNN "Packaging"
+F 12 "±1%" H 2550 2600 50  0001 C CNN "Tolerance"
+F 13 "0.063W, 1/16W" H 2550 2600 50  0001 C CNN "Power (Watts)"
+F 14 "Thick Film" H 2550 2600 50  0001 C CNN "Composition"
+F 15 "Automotive AEC-Q200, Moisture Resistant" H 2550 2600 50  0001 C CNN "Features"
+F 16 "±100ppm/°C" H 2550 2600 50  0001 C CNN "Temperature Coefficient"
+F 17 "-55°C ~ 155°C" H 2550 2600 50  0001 C CNN "Operating Temperature"
+F 18 "0402 (1005 Metric)" H 2550 2600 50  0001 C CNN "Package / Case"
+F 19 "AEC-Q200" H 2550 2600 50  0001 C CNN "Ratings"
+F 20 "0402" H 2550 2600 50  0001 C CNN "Supplier Device Package"
+F 21 "0.039\" L x 0.020\" W (1.00mm x 0.50mm)" H 2550 2600 50  0001 C CNN "Size / Dimension"
+F 22 "0.016\" (0.40mm)" H 2550 2600 50  0001 C CNN "Height - Seated (Max)"
+F 23 "2" H 2550 2600 50  0001 C CNN "Number of Terminations"
+F 24 "CRGCQ0402" H 2550 2600 50  0001 C CNN "Base Part Number"
+	1    2550 2600
+	1    0    0    -1
+$EndComp
+Wire Wire Line
+	2450 2450 2450 2400
+Connection ~ 2450 2400
+Wire Wire Line
+	2450 2400 2200 2400
+$Comp
+L Power:GND #PWR05
+U 1 1 60698399
+P 2450 2800
+F 0 "#PWR05" H 2450 2600 50  0001 C CNN
+F 1 "GND" H 2455 2662 50  0000 C CNN
+F 2 "" H 2450 2800 50  0001 C CNN
+F 3 "" H 2450 2800 50  0001 C CNN
+	1    2450 2800
+	1    0    0    -1
+$EndComp
+Wire Wire Line
+	2450 2750 2450 2800
 $EndSCHEMATC
