File: IR-Controller/hardware/IR-Controller.kicad_pcb (KiCad board)
At the start: 2 copper layers, 7 parts, among them Q1 MMBT3904LT1G, U1 PIC18LF2550-ISO

Commit message: Initial version of controller suitable for debugging
Parts:
- added J1: Conn_1x06_Generic, Connector_Generic:Conn_1x06_Socket_Pitch2.54mm_sideways, F.Cu at (183.2, 69.0)
- added R3: CRGCQ0402F10K, Resistor:R_0402_1005Metric, F.Cu at (157.4, 73.5)
- added SW1: MCSLPT4644B1TR, Switches:MCSLPT4644B1TR, F.Cu at (167.5, 92.1)
- added SW2: MCSLPT4644B1TR, Switches:MCSLPT4644B1TR, F.Cu at (167.5, 82.0)
- BT1, C1, D1, Q1, R1, R2, U1: moved to F.Cu
- moved D1 87.9 mm to (167.5, 58.0), turned to 180 degrees
- moved R1 86.3 mm to (164.5, 57.5), turned to 90 degrees
- moved BT1 85.0 mm to (167.5, 119.1)
- moved C1 83.0 mm to (154.9, 73.5), turned to 0 degrees
- moved Q1 82.1 mm to (161.8, 58.0), turned to 0 degrees
- moved U1 80.1 mm to (157.5, 66.9), turned to 270 degrees
- moved R2 76.6 mm to (157.9, 57.5)
Connections:
- net +3V0 renamed +3V
- U1 pad 1: Net-(U1-Pad1) -> /MCLR
- U1 pad 21: Net-(U1-Pad21) -> /SW_COL_0
- U1 pad 25: Net-(U1-Pad25) -> /SW_ROW_0
- U1 pad 26: Net-(U1-Pad26) -> /SW_ROW_1
- U1 pad 27: Net-(U1-Pad27) -> /PGC
- U1 pad 28: Net-(U1-Pad28) -> /PGD
Routing:
- net +3V: track 0.00 -> 112.1 mm
- net /SW_ROW_1: track 0.00 -> 38.1 mm
- net /SW_COL_0: track 0.00 -> 35.4 mm
- net GND: track 0.00 -> 28.6 mm
- net /SW_ROW_0: track 0.00 -> 27.5 mm
- net /PGC: track 0.00 -> 16.4 mm
- net /PGD: track 0.00 -> 13.5 mm
- net Net-(R2-Pad2): track 0.00 -> 10.3 mm
- net Net-(D1-Pad1): track 0.00 -> 6.28 mm
- net Net-(Q1-Pad1): track 0.00 -> 2.73 mm
- net Net-(Q1-Pad3): track 0.00 -> 1.55 mm
- added copper zone on F.Cu, net GND
Other:
- board outline added: 40.1 x 80.1 mm

Commit message: Controller: Pull MCLR to ground via 10k resistor
When MCLR is used the pin acts as an input. Pull to ground to avoid its
floating state. Use 10k resistor so that the ICSP can still work.

Also update the board.
Parts:
- added R3: CRGCQ0402F10K, Resistor:R_0402_1005Metric, F.Cu at (164.5, 60.3)
- renumbered R3 to R4
Connections:
- U1 pad 15: Net-(U1-Pad15) -> GND
- U1 pad 16: Net-(U1-Pad16) -> GND
Routing:
- net GND: track 28.6 -> 44.6 mm
- net /MCLR: track 0.00 -> 2.35 mm

Commit message: Controller: Allow sliding battery
The power track was causing an intermediate short circuit when
sliding battery in and out.
Routing:
- net +3V: track 112.1 -> 70.1 mm
Changed lines of the file:
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@@
     (thickness 1.6)
     (drawings 12)
-    (tracks 82)
+    (tracks 77)
     (zones 0)
     (modules 12)
@@
   (segment (start 155.575 69.596) (end 160.147 65.024) (width 0.508) (layer F.Cu) (net 21))
   (segment (start 155.575 71.501) (end 155.575 69.596) (width 0.508) (layer F.Cu) (net 21))
-  (segment (start 155.608 119.0625) (end 155.608 125.9535) (width 0.8128) (layer F.Cu) (net 21))
-  (segment (start 179.418 125.9535) (end 179.418 119.0625) (width 0.8128) (layer F.Cu) (net 21))
-  (segment (start 174.117 131.2545) (end 179.418 125.9535) (width 0.8128) (layer F.Cu) (net 21))
-  (segment (start 160.909 131.2545) (end 174.117 131.2545) (width 0.8128) (layer F.Cu) (net 21))
-  (segment (start 155.608 125.9535) (end 160.909 131.2545) (width 0.8128) (layer F.Cu) (net 21))
   (segment (start 165.388 93.825) (end 169.638 93.825) (width 0.6096) (layer F.Cu) (net 22))
   (segment (start 171.45 76.073) (end 174.5615 79.1845) (width 0.508) (layer F.Cu) (net 22))

Commit message: Update exports
Parts:
- moved BT1 17.2 mm to (150.4, 119.7)
- moved C1 17.2 mm to (137.8, 74.1)
- moved D1 17.2 mm to (150.4, 58.6)
- moved Q1 17.2 mm to (144.7, 58.6)
- moved R1 17.2 mm to (147.3, 58.2)
- moved R3 17.2 mm to (147.3, 61.0)
- moved R4 17.2 mm to (140.2, 74.1)
- moved SW1 17.2 mm to (150.4, 92.7)
- moved SW2 17.2 mm to (150.4, 82.7)
- moved J1 17.2 mm to (166.1, 69.6)
- moved R2 17.2 mm to (140.8, 58.2)
- moved U1 17.2 mm to (140.3, 67.6)
